File: pcb/TSC_board.kicad_pcb (KiCad board)
At the start: 4 copper layers, 160 x 100 mm, 187 parts, among them IC1 SN65HVD75DR, IC27 NL17SZ17DFT2G, IC28 NL17SZ17DFT2G, IC29 NL17SZ17DFT2G, IC30 NL17SZ17DFT2G, IC31 NL17SZ17DFT2G, IC32 NL17SZ17DFT2G, IC33 NL17SZ17DFT2G, IC34 NL17SZ17DFT2G, IC35 NL17SZ17DFT2G, IC36 NL17SZ17DFT2G, IC37 NL17SZ17DFT2G, IC38 NL17SZ17DFT2G, IC39 NL17SZ17DFT2G, IC40 NL17SZ17DFT2G, J1 DIN41612_02x32_AC, J2 TC2030, J3 Conn_01x02_Pin, T1 H1102NL, U1 W5500, U2 STM32G484METx, U27 ADuM1300xRW, U28 ADuM1300xRW, U29 TEA1-0505, U3 USBLC6-2SC6, U30 TEA1-0505, U31 TEA1-0505, U32 TEA1-0505, U4 USBLC6-2SC6, U5 USBLC6-2SC6, U6 FM24C64B, U7 ADuM1400xRW, U8 ADuM1400xRW, Y1 3225-25M-SR, Y2 3225-25M-SR

Commit message: Change of concept, only frontend. To be connected with UCB_board
Parts:
- removed C12, C13, C14, C15, C16, C17, C27, C28, C29, C32, C33, C34, C37, C38, C39, C41, C42, C45, C46, C49, C50, C52: 100n, Capacitor_SMD:C_0603_1608Metric_Pad1.08x0.95mm_HandSolder
- removed C18, C30, C31, C35, C36, C40, C43, C44, C47, C48, C51: 10u, Capacitor_SMD:C_1206_3216Metric_Pad1.33x1.80mm_HandSolder
- removed C19, C20: 18p, Capacitor_SMD:C_0402_1005Metric_Pad0.74x0.62mm_HandSolder
- removed C21, C22, C23, C24, C25, C53, C54, C65: 10n, Capacitor_SMD:C_0603_1608Metric_Pad1.08x0.95mm_HandSolder
- removed D10, D16, D17, D5: ESD5Z3.3T1G, Diode_SMD:D_SOD-523
- removed D11: D_TVS, Diode_SMD:D_MiniMELF
- removed D12, D7: SMF5.0CA, Diode_SMD:D_SMF
- removed D13, D14, D4, D6: ~, LED_SMD:LED_0603_1608Metric_Pad1.05x0.95mm_HandSolder
- removed D15: CDSOT23-SM712, SamacSys_Parts:SOT95P230X117-3N
- removed F1, F2: Polyfuse, Fuse:Fuse_1206_3216Metric_Pad1.42x1.75mm_HandSolder
- removed J2: TC2030, Connector:Tag-Connect_TC2030-IDC-NL_2x03_P1.27mm_Vertical
- removed J3: Conn_01x02_Pin, Connector_PinHeader_2.00mm:PinHeader_1x02_P2.00mm_Vertical
- removed JP1: SolderJumper_3_Bridged12, Jumper:SolderJumper-3_P1.3mm_Bridged12_Pad1.0x1.5mm
- removed L1: B82464P4105M000, Inductor_SMD:L_10.4x10.4_H4.8
- removed L2, L3, L4: LQH32PN101MN0L, Inductor_SMD:L_1210_3225Metric
- removed R17: 33R, Resistor_SMD:R_0603_1608Metric_Pad0.98x0.95mm_HandSolder
- removed R18, R20: 1M, Resistor_SMD:R_0402_1005Metric_Pad0.72x0.64mm_HandSolder
- removed R19: 12,4k, Resistor_SMD:R_0603_1608Metric_Pad0.98x0.95mm_HandSolder
- removed R21, R84, R85, R90, R91: 10k, Resistor_SMD:R_0603_1608Metric_Pad0.98x0.95mm_HandSolder
- removed R76, R77, R78, R79, R86, R87: 120, Resistor_SMD:R_0603_1608Metric_Pad0.98x0.95mm_HandSolder
- removed R80: 0R, Resistor_SMD:R_0402_1005Metric_Pad0.72x0.64mm_HandSolder
- removed R88, R89: 10R, Resistor_SMD:R_0603_1608Metric_Pad0.98x0.95mm_HandSolder
- removed RN1, RN2, RN3: 4x10k, Resistor_SMD:R_Array_Convex_4x0603
- removed T1: H1102NL, SamacSys_Parts:SOIC127P940X597-16N
- removed TP1, TP12, TP13, TP14, TP15, TP16, TP17, TP18, TP19, TP2, TP20, TP21, TP22, TP3, TP4, TP5, TP6, TP7, TP8: TestPoint, TestPoint:TestPoint_Pad_D1.0mm
- removed U5: USBLC6-2SC6, Package_TO_SOT_SMD:SOT-23-6_Handsoldering
- removed U6: FM24C64B, Package_SO:SOIC-8_3.9x4.9mm_P1.27mm
- removed Y1, Y2: 3225-25M-SR, Crystal:Crystal_SMD_3225-4Pin_3.2x2.5mm
- added IC2: TS3021ILT, TS3021ILT:SOT95P280X145-5N, F.Cu at (92.8, -67.3)
- added IC3: TS3021ILT, TS3021ILT:SOT95P280X145-5N, F.Cu at (92.8, -62.8)
- added IC4: TS3021ILT, TS3021ILT:SOT95P280X145-5N, F.Cu at (92.8, -58.2)
- C3: value 1nF/2kV -> 100n; footprint Capacitor_SMD:C_1206_3216Metric_Pad1.33x1.80mm_HandSolder -> Capacitor_SMD:C_0603_1608Metric_Pad1.08x0.95mm_HandSolder
- C4: value 10n -> 100n
- C5: value 1nF/2kV -> 100n
- C6: value 18p -> 100n; footprint Capacitor_SMD:C_0402_1005Metric_Pad0.74x0.62mm_HandSolder -> Capacitor_SMD:C_0603_1608Metric_Pad1.08x0.95mm_HandSolder
- C7: value 10n -> 1n
- C8: value 18p -> 10u; footprint Capacitor_SMD:C_0402_1005Metric_Pad0.74x0.62mm_HandSolder -> Capacitor_SMD:C_1206_3216Metric
- C9: value 4,7u -> 10u; footprint Capacitor_SMD:C_0603_1608Metric_Pad1.08x0.95mm_HandSolder -> Capacitor_SMD:C_1206_3216Metric
- D1, D2: value ~ -> SMF5.0CA; footprint LED_SMD:LED_0603_1608Metric_Pad1.05x0.95mm_HandSolder -> Diode_SMD:D_SMF
- D3: value ESD5Z3.3T1G -> SMF5.0CA; footprint Diode_SMD:D_SOD-523 -> Diode_SMD:D_SMF
- IC1: value SN65HVD75DR -> TS3021ILT; footprint SamacSys_Parts:SOIC127P600X175-8N -> TS3021ILT:SOT95P280X145-5N
- R1: value 22R -> 10k; footprint Resistor_SMD:R_0402_1005Metric_Pad0.72x0.64mm_HandSolder -> Resistor_SMD:R_0603_1608Metric
- R10: value 49R9 -> 10k; footprint Resistor_SMD:R_0603_1608Metric_Pad0.98x0.95mm_HandSolder -> Resistor_SMD:R_0603_1608Metric
- R11: value 49R9 -> 100; footprint Resistor_SMD:R_0603_1608Metric_Pad0.98x0.95mm_HandSolder -> Resistor_SMD:R_0603_1608Metric
- R12: value 150R -> 100k; footprint Resistor_SMD:R_0603_1608Metric_Pad0.98x0.95mm_HandSolder -> Resistor_SMD:R_0603_1608Metric
- R13: value 150R -> 0R; footprint Resistor_SMD:R_0603_1608Metric_Pad0.98x0.95mm_HandSolder -> Resistor_SMD:R_0402_1005Metric
- R14, R15, R16: value 33R -> 0R; footprint Resistor_SMD:R_0603_1608Metric_Pad0.98x0.95mm_HandSolder -> Resistor_SMD:R_0402_1005Metric
- R2: value 22R -> 100k; footprint Resistor_SMD:R_0402_1005Metric_Pad0.72x0.64mm_HandSolder -> Resistor_SMD:R_0603_1608Metric
- R3: value 10k -> 100; footprint Resistor_SMD:R_0603_1608Metric_Pad0.98x0.95mm_HandSolder -> Resistor_SMD:R_0603_1608Metric
- R4: value 15k -> 10k; footprint Resistor_SMD:R_0603_1608Metric_Pad0.98x0.95mm_HandSolder -> Resistor_SMD:R_0603_1608Metric
- R5: value 10R -> 100; footprint Resistor_SMD:R_0603_1608Metric_Pad0.98x0.95mm_HandSolder -> Resistor_SMD:R_0603_1608Metric
- R6: value 75R -> 100k; footprint Resistor_SMD:R_0603_1608Metric_Pad0.98x0.95mm_HandSolder -> Resistor_SMD:R_0603_1608Metric
- R7: value 75R -> 10k; footprint Resistor_SMD:R_0603_1608Metric_Pad0.98x0.95mm_HandSolder -> Resistor_SMD:R_0603_1608Metric
- R8: value 82R -> 100; footprint Resistor_SMD:R_0603_1608Metric_Pad0.98x0.95mm_HandSolder -> Resistor_SMD:R_0603_1608Metric
- R9: value 82R -> 100k; footprint Resistor_SMD:R_0603_1608Metric_Pad0.98x0.95mm_HandSolder -> Resistor_SMD:R_0603_1608Metric
- U1: value W5500 -> DAC7311xDCK; footprint Package_QFP:LQFP-48_7x7mm_P0.5mm -> Package_TO_SOT_SMD:SOT-363_SC-70-6
- U3: value USBLC6-2SC6 -> ADuM1300xRW; footprint Package_TO_SOT_SMD:SOT-23-6_Handsoldering -> Package_SO:SOIC-16W_7.5x10.3mm_P1.27mm
- U4: value USBLC6-2SC6 -> LM4040DBZ-5; footprint Package_TO_SOT_SMD:SOT-23-6_Handsoldering -> Package_TO_SOT_SMD:SOT-23
- moved R13 249.8 mm to (106.8, -82.6), turned to -15 degrees
- moved R12 245.4 mm to (97.8, -76.0)
- moved R6 245.4 mm to (97.8, -74.5)
- moved R7 245.4 mm to (97.8, -80.8)
Connections:
- C1 pad 1: +5V -> Net-(IC27-GND)
- C1 pad 2: GND -> Net-(IC27-VCC)
- C10 pad 2: Net-(U1-1V2O) -> +3.3V
- C11 pad 1: GND -> +3.3V
- C11 pad 2: +3.3V -> GND
- C2 pad 1: +5V -> Net-(U1-AVDD/AVREF)
- C2 pad 2: GND -> Net-(IC27-GND)
- C26 pad 1: +3.3V -> Net-(C26-Pad1)
- C26 pad 2: GND -> Net-(C26-Pad2)
- C3 pad 1: Earth -> Net-(IC1-VCC+)
- C3 pad 2: GND -> Net-(D33-A2)
- C4 pad 1: GND -> Net-(IC2-VCC+)
- C4 pad 2: Net-(T1-CT_1) -> Net-(D1-A2)
- C5 pad 1: Net-(C5-Pad1) -> Net-(IC3-VCC+)
- C5 pad 2: Earth -> Net-(D2-A2)
- C55 pad 1: GND -> Net-(C26-Pad2)
- C55 pad 2: +3.3V -> Net-(C26-Pad1)
- C6 pad 1: /EthernetPHY/XO+ -> Net-(IC4-VCC+)
- C6 pad 2: GND -> Net-(D3-A2)
- C7 pad 1: Net-(T1-CT_2) -> Net-(U1-VOUT)
- C7 pad 2: GND -> Net-(IC27-GND)
- C8 pad 1: /EthernetPHY/XO- -> Net-(IC27-VCC)
- C8 pad 2: GND -> Net-(IC27-GND)
- C9 pad 1: Net-(U1-TOCAP) -> +5V
- D1 pad 1: Net-(D1-K) -> Net-(D1-A1)
- D1 pad 2: /EthernetPHY/SPEED -> Net-(D1-A2)
- D2 pad 1: Net-(D2-K) -> Net-(D2-A1)
- D2 pad 2: /EthernetPHY/LINK -> Net-(D2-A2)
- D3 pad 1: /ConnectorDIN41612/USART+ -> Net-(D3-A1)
- D3 pad 2: GND -> Net-(D3-A2)
- D33 pad 1: unconnected-(D33-A1-Pad1) -> Net-(D33-A1)
- D33 pad 2: unconnected-(D33-A2-Pad2) -> Net-(D33-A2)
- IC1 pad 1: /ConnectorDIN41612/RxD -> Net-(IC1-OUT)
- IC1 pad 2: /ConnectorDIN41612/DE -> Net-(D33-A2)
- IC1 pad 3: /ConnectorDIN41612/DE -> Net-(IC1-IN+)
- IC1 pad 4: /ConnectorDIN41612/TxD -> Net-(IC1-IN-)
- IC1 pad 5: GND -> Net-(IC1-VCC+)
- IC27 pad 2: unconnected-(IC27-A-Pad2) -> Net-(IC1-OUT)
- IC28 pad 2: unconnected-(IC28-A-Pad2) -> Net-(IC2-OUT)
- IC29 pad 2: unconnected-(IC29-A-Pad2) -> Net-(IC29-A)
- IC30 pad 2: unconnected-(IC30-A-Pad2) -> Net-(IC30-A)
- R1 pad 1: /ConnectorDIN41612/USB_D+ -> Net-(D33-A1)
- R1 pad 2: /ConnectorDIN41612/USB_DP -> Net-(IC1-IN+)
- R10 pad 1: +3.3V -> Net-(D3-A1)
- R10 pad 2: /ConnectorDIN41612/TD+ -> Net-(IC4-IN+)
- R11 pad 1: +3.3V -> Net-(U1-VOUT)
- R11 pad 2: /ConnectorDIN41612/TD- -> Net-(IC4-IN-)
- R12 pad 1: /ConnectorDIN41612/RX+ -> Net-(IC4-IN+)
- R12 pad 2: Net-(C5-Pad1) -> Net-(IC30-A)
- R13 pad 1: /ConnectorDIN41612/RX- -> Net-(IC1-OUT)
- R13 pad 2: Net-(C5-Pad1) -> Net-(IC27-Y)
- R14 pad 1: /EthernetPHY/TXN -> Net-(IC2-OUT)
- R14 pad 2: /ConnectorDIN41612/ETH_TD- -> Net-(IC28-Y)
- R15 pad 1: /EthernetPHY/TXP -> Net-(IC29-A)
- R15 pad 2: /ConnectorDIN41612/ETH_TD+ -> Net-(IC29-Y)
- R16 pad 1: /EthernetPHY/RXN -> Net-(IC30-A)
- R16 pad 2: /ConnectorDIN41612/ETH_RD- -> Net-(IC30-Y)
- R2 pad 1: /ConnectorDIN41612/USB_D- -> Net-(IC1-IN+)
- R2 pad 2: /ConnectorDIN41612/USB_DN -> Net-(IC1-OUT)
- R3 pad 1: /ConnectorDIN41612/USB_DET -> Net-(U1-VOUT)
- R3 pad 2: /ConnectorDIN41612/VUSB -> Net-(IC1-IN-)
- R4 pad 1: GND -> Net-(D1-A1)
- R4 pad 2: /ConnectorDIN41612/USB_DET -> Net-(IC2-IN+)
- R5 pad 1: +3.3V -> Net-(U1-VOUT)
- R5 pad 2: Net-(T1-CT_1) -> Net-(IC2-IN-)
- R6 pad 1: Net-(T1-NC_3) -> Net-(IC2-IN+)
- R6 pad 2: Net-(C5-Pad1) -> Net-(IC2-OUT)
- R7 pad 1: Net-(T1-NC_6) -> Net-(D2-A1)
- R7 pad 2: Net-(C5-Pad1) -> Net-(IC3-IN+)
- R8 pad 1: /ConnectorDIN41612/RD+ -> Net-(U1-VOUT)
- R8 pad 2: Net-(T1-CT_2) -> Net-(IC3-IN-)
- R9 pad 1: /ConnectorDIN41612/RD- -> Net-(IC3-IN+)
- R9 pad 2: Net-(T1-CT_2) -> Net-(IC29-A)
- U1 pad 1: /EthernetPHY/TXN -> Net-(U1-~{SYNC})
- U1 pad 2: /EthernetPHY/TXP -> Net-(U1-SCLK)
- U1 pad 3: GND -> Net-(U1-DIN)
- U1 pad 4: +3.3V -> Net-(U1-AVDD/AVREF)
- U1 pad 5: /EthernetPHY/RXN -> Net-(IC27-GND)
- U1 pad 6: /EthernetPHY/RXP -> Net-(U1-VOUT)
- U2 pad 1: +3.3V -> unconnected-(U2-VBAT-Pad1)
- U2 pad 15: GND -> Net-(U2-VSS-Pad15)
- U2 pad 16: +3.3V -> unconnected-(U2-VDD-Pad16)
- U2 pad 25: /MCU/LED_R -> unconnected-(U2-PB1-Pad25)
- U2 pad 26: /MCU/LED_G -> unconnected-(U2-PB2-Pad26)
- U2 pad 27: GND -> unconnected-(U2-VSSA-Pad27)
- U2 pad 28: +3.3V -> unconnected-(U2-VREF+-Pad28)
- U2 pad 29: +3.3V -> unconnected-(U2-VDDA-Pad29)
- U2 pad 33: /MCU/QSPI_CLK -> unconnected-(U2-PE10-Pad33)
- U2 pad 34: /MCU/QSPI_NCS -> unconnected-(U2-PE11-Pad34)
- U2 pad 35: /MCU/QSPI_IO0 -> unconnected-(U2-PE12-Pad35)
- U2 pad 36: /MCU/QSPI_IO1 -> unconnected-(U2-PE13-Pad36)
- U2 pad 37: /MCU/QSPI_IO2 -> unconnected-(U2-PE14-Pad37)
- U2 pad 38: /MCU/QSPI_IO3 -> unconnected-(U2-PE15-Pad38)
- U2 pad 40: GND -> Net-(U2-VSS-Pad15)
- U2 pad 41: +3.3V -> unconnected-(U2-VDD-Pad41)
- U2 pad 44: /EthernetPHY/SCK -> unconnected-(U2-PB13-Pad44)
- U2 pad 45: /EthernetPHY/MISO -> unconnected-(U2-PB14-Pad45)
- U2 pad 46: /EthernetPHY/MOSI -> unconnected-(U2-PB15-Pad46)
- U2 pad 47: /EthernetPHY/CS -> unconnected-(U2-PD8-Pad47)
- U2 pad 48: /EthernetPHY/RST -> unconnected-(U2-PD9-Pad48)
- U2 pad 49: /EthernetPHY/INT -> unconnected-(U2-PD10-Pad49)
- U2 pad 5: /MCU/XTAL+ -> unconnected-(U2-PF0-Pad5)
- U2 pad 50: GND -> Net-(U2-VSS-Pad15)
- U2 pad 51: +3.3V -> unconnected-(U2-VDD-Pad51)
- U2 pad 54: /MCU/SCL -> unconnected-(U2-PC8-Pad54)
- U2 pad 55: /MCU/SDA -> unconnected-(U2-PC9-Pad55)
- U2 pad 56: /EthernetPHY/CLKIN -> unconnected-(U2-PA8-Pad56)
- U2 pad 57: /ConnectorDIN41612/USART+ -> unconnected-(U2-PA9-Pad57)
- U2 pad 58: /ConnectorDIN41612/USART- -> unconnected-(U2-PA10-Pad58)
- U2 pad 59: /ConnectorDIN41612/USB_D- -> unconnected-(U2-PA11-Pad59)
- U2 pad 6: /MCU/XTAL- -> unconnected-(U2-PF1-Pad6)
- U2 pad 60: /ConnectorDIN41612/USB_D+ -> unconnected-(U2-PA12-Pad60)
- U2 pad 61: GND -> Net-(U2-VSS-Pad15)
- U2 pad 62: +3.3V -> unconnected-(U2-VDD-Pad62)
- U2 pad 63: /MCU/SWDIO -> unconnected-(U2-PA13-Pad63)
- U2 pad 64: /MCU/SWCLK -> unconnected-(U2-PA14-Pad64)
- U2 pad 65: /ConnectorDIN41612/DE -> unconnected-(U2-PA15-Pad65)
- U2 pad 66: /ConnectorDIN41612/TxD -> unconnected-(U2-PC10-Pad66)
- U2 pad 67: /ConnectorDIN41612/RxD -> unconnected-(U2-PC11-Pad67)
- U2 pad 69: /ConnectorDIN41612/USB_DET -> unconnected-(U2-PD0-Pad69)
- U2 pad 7: /MCU/nRESET -> unconnected-(U2-PG10-Pad7)
- U2 pad 72: /MCU/SWO -> unconnected-(U2-PB3-Pad72)
- U2 pad 77: /MCU/BOOT -> unconnected-(U2-PB8-Pad77)
- U2 pad 79: GND -> Net-(U2-VSS-Pad15)
- U2 pad 80: +3.3V -> unconnected-(U2-VDD-Pad80)
- U3 pad 1: /ConnectorDIN41612/USB_DP -> +3.3V
- U3 pad 3: /ConnectorDIN41612/USB_DN -> unconnected-(U3-V_{IA}-Pad3)
- U3 pad 4: /ConnectorDIN41612/D- -> unconnected-(U3-V_{IB}-Pad4)
- U3 pad 5: /ConnectorDIN41612/VUSB -> unconnected-(U3-V_{IC}-Pad5)
- U3 pad 6: /ConnectorDIN41612/D+ -> unconnected-(U3-NC-Pad6)
- U4 pad 1: /ConnectorDIN41612/ETH_TD- -> Net-(U1-AVDD/AVREF)
- U4 pad 2: GND -> Net-(IC27-GND)
- U4 pad 3: /ConnectorDIN41612/ETH_TD+ -> unconnected-(U4-NC-Pad3)
Routing:
- added copper zone on B.Cu, net (none)
- added copper zone on F.Cu, net (none)
- removed copper zone on F.Cu, net Net-(C27-Pad1)
- removed copper zone on B.Cu, net Net-(D11-A2)
- removed copper zone on F.Cu, net Net-(D11-A2)

Commit message: Add STM32 .ioc and adjust UCB connector footprint
Add STM32CubeMX project file (firmware/TSC_board.ioc) for the STM32H563VITx MCU and update KiCad PCB/schematic files. Adjust UCB_conn footprint and apply corresponding changes to pcb TSC_board/Frontend/MCU schematic and project files to reflect the connector/placement updates.
Parts:
- removed C56, C58, C60, C62, C64, C68: 10n, Capacitor_SMD:C_0603_1608Metric_Pad1.08x0.95mm_HandSolder
- removed C57, C59, C61, C63, C66, C70: 100n, Capacitor_SMD:C_0603_1608Metric_Pad1.08x0.95mm_HandSolder
- removed IC31, IC32, IC33, IC34, IC35, IC36, IC37, IC38, IC39, IC40: NL17SZ17DFT2G, SamacSys_Parts:SOT65P210X110-5N
- removed U2: STM32G484METx, Package_QFP:LQFP-80_12x12mm_P0.5mm
- removed U27, U28: ADuM1300xRW, Package_SO:SOIC-16W_7.5x10.3mm_P1.27mm
- removed U30, U31, U32: TEA1-0505, Converter_DCDC:Converter_DCDC_TRACO_TEA1-xxxx_THT
- removed U7: ADuM1400xRW, Package_SO:SOIC-16W_7.5x10.3mm_P1.27mm
- added C12: 100n, Capacitor_SMD:C_0603_1608Metric, F.Cu at (68.6, -33.6)
- added FB1: 100R @ 100MHz, Inductor_SMD:L_0603_1608Metric, F.Cu at (48.0, -61.0)
- added FB2: 100R @ 100MHz, Inductor_SMD:L_0603_1608Metric, F.Cu at (76.5, -80.3)
- added FB3: 100R @ 100MHz, Inductor_SMD:L_0603_1608Metric, F.Cu at (76.5, -77.8)
- added FB4: 100R @ 100MHz, Inductor_SMD:L_0603_1608Metric, F.Cu at (76.5, -75.3)
- added FB5: 100R @ 100MHz, Inductor_SMD:L_0603_1608Metric, F.Cu at (76.5, -72.8)
- added FB6: 100R @ 100MHz, Inductor_SMD:L_0603_1608Metric, F.Cu at (162.6, 61.0)
- added FB7: 100R @ 100MHz, Inductor_SMD:L_0603_1608Metric, F.Cu at (162.6, 63.0)
- added FB8: 100R @ 100MHz, Inductor_SMD:L_0603_1608Metric, F.Cu at (162.6, 65.0)
- added FB9: 100R @ 100MHz, Inductor_SMD:L_0603_1608Metric, F.Cu at (162.6, 67.0)
- added J2: Conn_01x05_Socket, Connector_Phoenix_MC:PhoenixContact_MC_1,5_5-G-3.5_1x05_P3.50mm_Horizontal, F.Cu at (43.1, 84.1)
- added J3: Conn_01x04_Socket, Connector_Phoenix_MC:PhoenixContact_MC_1,5_4-G-3.5_1x04_P3.50mm_Horizontal, F.Cu at (43.1, 104.7)
- added J4: Conn_01x04_Socket, Connector_Phoenix_MC:PhoenixContact_MC_1,5_4-G-3.5_1x04_P3.50mm_Horizontal, F.Cu at (43.1, 121.7)
- added R17: 330R, Resistor_SMD:R_0603_1608Metric, F.Cu at (46.5, -61.0)
- added X1: ~, Conn:UCB_conn, F.Cu at (170.0, 100.0)
- C1, C10, C2, C4, C6, C67, C69, C7, C71: footprint Capacitor_SMD:C_0603_1608Metric_Pad1.08x0.95mm_HandSolder -> Capacitor_SMD:C_0603_1608Metric
- C11, C3: footprint Capacitor_SMD:C_0603_1608Metric_Pad1.08x0.95mm_HandSolder -> Capacitor_SMD:C_0603_1608Metric; moved to F.Cu
- C26: footprint Capacitor_SMD:C_1206_3216Metric_Pad1.33x1.80mm_HandSolder -> Capacitor_SMD:C_1206_3216Metric
- C5: footprint Capacitor_SMD:C_1206_3216Metric_Pad1.33x1.80mm_HandSolder -> Capacitor_SMD:C_0603_1608Metric
- C55: value 10n -> 100n; footprint Capacitor_SMD:C_0603_1608Metric_Pad1.08x0.95mm_HandSolder -> Capacitor_SMD:C_0603_1608Metric
- J1: value DIN41612_02x32_AC -> Conn_01x05_Socket; footprint Connector_DIN:DIN41612_C_2x32_Male_Horizontal_THT -> Connector_Phoenix_MC:PhoenixContact_MC_1,5_5-G-3.5_1x05_P3.50mm_Horizontal
- moved C7 254.0 mm to (43.3, -60.8)
- moved R16 249.3 mm to (40.9, -64.1), turned to 0 degrees
- moved R14 249.0 mm to (40.9, -68.1)
- moved R15 248.7 mm to (40.9, -66.1)
- moved C2 247.6 mm to (45.0, -60.8), turned to 90 degrees
- moved U4 240.9 mm to (47.5, -57.6)
- moved U1 237.2 mm to (44.1, -57.4), turned to 90 degrees
- moved C3 237.2 mm to (64.3, -38.6), turned to 0 degrees
- moved C5 235.4 mm to (64.3, -33.6)
- moved R11 234.5 mm to (72.1, -58.7), turned to 0 degrees
- moved R10 233.0 mm to (72.1, -61.2), turned to 0 degrees
- moved R5 231.3 mm to (68.1, -56.2), turned to 0 degrees
- moved U3 231.1 mm to (55.7, -56.9), turned to 180 degrees
- moved R9 230.6 mm to (68.1, -46.2), turned to 0 degrees
- moved R8 230.3 mm to (68.1, -48.7), turned to 0 degrees
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Connections:
- C1 pad 1: Net-(IC27-GND) -> Net-(U1-GND)
- C2 pad 2: Net-(IC27-GND) -> Net-(U1-GND)
- C7 pad 2: Net-(IC27-GND) -> Net-(U1-GND)
- C8 pad 2: Net-(IC27-GND) -> Net-(U1-GND)
- U1 pad 5: Net-(IC27-GND) -> Net-(U1-GND)
- U29 pad 3: Net-(IC27-GND) -> Net-(U1-GND)
- U3 pad 15: Net-(IC27-GND) -> Net-(U1-GND)
- U3 pad 3: unconnected-(U3-V_{IA}-Pad3) -> /Frontend/MOSI
- U3 pad 4: unconnected-(U3-V_{IB}-Pad4) -> /Frontend/SCK
- U3 pad 5: unconnected-(U3-V_{IC}-Pad5) -> /Frontend/CS1
- U3 pad 9: Net-(IC27-GND) -> Net-(U1-GND)
- U4 pad 2: Net-(IC27-GND) -> Net-(U1-GND)
- U8 pad 2: Net-(IC27-GND) -> Net-(U1-GND)
- U8 pad 8: Net-(IC27-GND) -> Net-(U1-GND)
Routing:
- net Earth: track 118.9 -> 0.00 mm, vias 2 -> 0
- net Net-(U1-DIN): track 0.00 -> 11.8 mm
- net Net-(U1-~{SYNC}): track 0.00 -> 9.31 mm
- net Net-(U1-GND): track 0.00 -> 8.38 mm, vias 0 -> 1
- net Net-(U1-SCLK): track 0.00 -> 8.27 mm
- net Net-(U1-AVDD/AVREF): track 0.00 -> 5.51 mm
- net /ConnectorDIN41612/TX+: track 3.44 -> 0.00 mm
- net Net-(U1-VOUT): track 0.00 -> 1.71 mm
- net Net-(FB1-Pad1): track 0.00 -> 1.57 mm
- removed copper zone on B.Cu, net (none)
- removed copper zone on F.Cu, net (none)
- removed copper zone on F.Cu, net +3.3V
Other:
- board size 160 x 100 mm -> 100 x 100 mm
- board text removed: "BOOT"

Commit message: More schematic
Parts:
- removed C26: 10u, Capacitor_SMD:C_1206_3216Metric
- removed C55, C67, C71: 100n, Capacitor_SMD:C_0603_1608Metric
- removed C69: 10n, Capacitor_SMD:C_0603_1608Metric
- removed D33: SMF5.0CA, Diode_SMD:D_SMF
- removed U29: TEA1-0505, Converter_DCDC:Converter_DCDC_TRACO_TEA1-xxxx_THT
- removed U8: ADuM1400xRW, Package_SO:SOIC-16W_7.5x10.3mm_P1.27mm
- added C13: 10u, Capacitor_SMD:C_1206_3216Metric, F.Cu at (90.7, -41.8)
- added C14: 10n, Capacitor_SMD:C_0603_1608Metric, F.Cu at (68.6, -52.1)
- added C18: 100n, Capacitor_SMD:C_0603_1608Metric, F.Cu at (72.6, -72.2)
- added C19: 100n, Capacitor_SMD:C_0603_1608Metric, F.Cu at (72.6, -69.7)
- added C20: 10n, Capacitor_SMD:C_0603_1608Metric, F.Cu at (72.6, -67.2)
- added C25: 100n, Capacitor_SMD:C_0603_1608Metric, F.Cu at (72.6, -64.7)
- added C31: 100n, Capacitor_SMD:C_0603_1608Metric, F.Cu at (48.9, -73.9)
- added C32: 100n, Capacitor_SMD:C_0603_1608Metric, F.Cu at (55.1, -67.4)
- added C33: 100n, Capacitor_SMD:C_0603_1608Metric, F.Cu at (55.1, -64.9)
- added C34: 100n, Capacitor_SMD:C_0603_1608Metric, F.Cu at (55.1, -62.4)
- added D4: SMF5.0CA, Diode_SMD:D_SMF, F.Cu at (90.8, -48.5)
- added FB10: 100R @ 100MHz, Inductor_SMD:L_0603_1608Metric, F.Cu at (76.6, -72.2)
- added FB11: 100R @ 100MHz, Inductor_SMD:L_0603_1608Metric, F.Cu at (76.6, -69.7)
- added FB12: 100R @ 100MHz, Inductor_SMD:L_0603_1608Metric, F.Cu at (51.6, -73.4)
- added FB13: 100R @ 100MHz, Inductor_SMD:L_0603_1608Metric, F.Cu at (51.6, -70.7)
- added FB14: 100R @ 100MHz, Inductor_SMD:L_0603_1608Metric, F.Cu at (51.6, -67.9)
- added FB15: 100R @ 100MHz, Inductor_SMD:L_0603_1608Metric, F.Cu at (51.6, -65.2)
- added R18: 10k, Resistor_SMD:R_0603_1608Metric, F.Cu at (-20.1, -80.5)
- added R19: 10k, Resistor_SMD:R_0603_1608Metric, F.Cu at (-20.2, -78.1)
- added R20: 10k, Resistor_SMD:R_0603_1608Metric, F.Cu at (-20.2, -75.5)
- added R21: 10k, Resistor_SMD:R_0603_1608Metric, F.Cu at (-20.2, -73.0)
- added R22: 10k, Resistor_SMD:R_0603_1608Metric, F.Cu at (-20.2, -70.5)
- added R23: 10k, Resistor_SMD:R_0603_1608Metric, F.Cu at (-20.2, -68.0)
- added R24: 10k, Resistor_SMD:R_0603_1608Metric, F.Cu at (-20.2, -65.5)
- added R25: 10k, Resistor_SMD:R_0603_1608Metric, F.Cu at (-20.2, -63.0)
- added R26: 10k, Resistor_SMD:R_0603_1608Metric, F.Cu at (-19.9, -60.4)
- added R27: 10k, Resistor_SMD:R_0603_1608Metric, F.Cu at (-16.2, -80.6)
- added R28: 10k, Resistor_SMD:R_0603_1608Metric, F.Cu at (-16.2, -78.1)
- added R29: 10k, Resistor_SMD:R_0603_1608Metric, F.Cu at (-16.2, -75.5)
- added R30: 10k, Resistor_SMD:R_0603_1608Metric, F.Cu at (-16.2, -73.0)
- added R31: 10k, Resistor_SMD:R_0603_1608Metric, F.Cu at (-16.2, -70.5)
- added R32: 10k, Resistor_SMD:R_0603_1608Metric, F.Cu at (-16.2, -68.0)
- added R33: 10k, Resistor_SMD:R_0603_1608Metric, F.Cu at (-16.2, -65.5)
- added R34: 10k, Resistor_SMD:R_0603_1608Metric, F.Cu at (-16.2, -63.0)
- added R35: 10k, Resistor_SMD:R_0603_1608Metric, F.Cu at (-16.2, -60.5)
- added R36: 10k, Resistor_SMD:R_0603_1608Metric, F.Cu at (-12.1, -80.6)
- added R37: 10k, Resistor_SMD:R_0603_1608Metric, F.Cu at (-12.2, -78.1)
- added R38: 10k, Resistor_SMD:R_0603_1608Metric, F.Cu at (-18.1, -90.0)
- added R39: 10k, Resistor_SMD:R_0603_1608Metric, F.Cu at (-11.9, -50.4)
- added R40: 10k, Resistor_SMD:R_0603_1608Metric, F.Cu at (-12.1, -70.5)
- added R41: 10k, Resistor_SMD:R_0603_1608Metric, F.Cu at (-12.1, -68.0)
- added R42: 10k, Resistor_SMD:R_0603_1608Metric, F.Cu at (-12.1, -65.5)
- added R43: 10k, Resistor_SMD:R_0603_1608Metric, F.Cu at (-12.1, -63.0)
- added R44: 10k, Resistor_SMD:R_0603_1608Metric, F.Cu at (-12.1, -60.5)
- added R45: 10k, Resistor_SMD:R_0603_1608Metric, F.Cu at (-8.13, -80.6)
- added R46: 10k, Resistor_SMD:R_0603_1608Metric, F.Cu at (-8.13, -78.1)
- added R47: 10k, Resistor_SMD:R_0603_1608Metric, F.Cu at (-8.13, -75.5)
- added R48: 10k, Resistor_SMD:R_0603_1608Metric, F.Cu at (-8.13, -73.0)
- added R49: 10k, Resistor_SMD:R_0603_1608Metric, F.Cu at (-8.13, -70.5)
- added R50: 470, Resistor_SMD:R_0603_1608Metric, F.Cu at (-8.13, -68.0)
- added R51: 470, Resistor_SMD:R_0603_1608Metric, F.Cu at (-12.7, -52.7)
- added R52: 470, Resistor_SMD:R_0603_1608Metric, F.Cu at (-38.6, -75.9)
- added R53: 470, Resistor_SMD:R_0603_1608Metric, F.Cu at (-38.6, -64.6)
- added R54: 470, Resistor_SMD:R_0603_1608Metric, F.Cu at (-4.12, -80.6)
- added R55: 470, Resistor_SMD:R_0603_1608Metric, F.Cu at (-38.6, -59.0)
- added R56: 470, Resistor_SMD:R_0603_1608Metric, F.Cu at (-4.12, -75.5)
- added R57: 470, Resistor_SMD:R_0603_1608Metric, F.Cu at (-4.12, -73.0)
- added R58: 470, Resistor_SMD:R_0603_1608Metric, F.Cu at (-4.12, -70.5)
- added R59: 470, Resistor_SMD:R_0603_1608Metric, F.Cu at (-30.1, -64.6)
- added R60: 470, Resistor_SMD:R_0603_1608Metric, F.Cu at (-30.1, -70.3)
- added R61: 470, Resistor_SMD:R_0603_1608Metric, F.Cu at (-26.1, -54.2)
- added U13: GAQY212GS, Package_SO:SOP-4_3.8x4.1mm_P2.54mm, F.Cu at (-13.6, -90.3)
- added U14: GAQY212GS, Package_SO:SOP-4_3.8x4.1mm_P2.54mm, F.Cu at (-34.9, -73.3)
- added U15: GAQY212GS, Package_SO:SOP-4_3.8x4.1mm_P2.54mm, F.Cu at (-34.9, -67.7)
- added U16: GAQY212GS, Package_SO:SOP-4_3.8x4.1mm_P2.54mm, F.Cu at (-34.9, -62.0)
- added U17: GAQY212GS, Package_SO:SOP-4_3.8x4.1mm_P2.54mm, F.Cu at (-34.9, -56.4)
- added U18: GAQY212GS, Package_SO:SOP-4_3.8x4.1mm_P2.54mm, F.Cu at (-34.9, -50.8)
- added U19: GAQY212GS, Package_SO:SOP-4_3.8x4.1mm_P2.54mm, F.Cu at (-26.4, -79.0)
- added U2: DAC7311xDCK, Package_TO_SOT_SMD:SOT-363_SC-70-6, F.Cu at (49.6, -45.0)
- added U21: GAQY212GS, Package_SO:SOP-4_3.8x4.1mm_P2.54mm, F.Cu at (-26.4, -73.3)
- added U22: GAQY212GS, Package_SO:SOP-4_3.8x4.1mm_P2.54mm, F.Cu at (-26.4, -67.7)
- added U23: GAQY212GS, Package_SO:SOP-4_3.8x4.1mm_P2.54mm, F.Cu at (-26.4, -62.0)
- added U24: GAQY212GS, Package_SO:SOP-4_3.8x4.1mm_P2.54mm, F.Cu at (-22.4, -51.6)
- added U5: ADuM1300xRW, Package_SO:SOIC-16W_7.5x10.3mm_P1.27mm, F.Cu at (73.0, -44.8)
- added U6: TEA1-0505, Converter_DCDC:Converter_DCDC_TRACO_TEA1-xxxx_THT, F.Cu at (84.6, -70.7)
- C10: value 10n -> 100n
- C11, C2: value 100n -> 10u; footprint Capacitor_SMD:C_0603_1608Metric -> Capacitor_SMD:C_1206_3216Metric
- C8, C9: value 10u -> 100n; footprint Capacitor_SMD:C_1206_3216Metric -> Capacitor_SMD:C_0603_1608Metric
- R1, R7: value 10k -> 1k
- R10: value 10k -> 50k
- R11: value 100 -> 50k
- R12, R9: value 100k -> 50k
- R2, R6: value 100k -> 100
- R3, R5: value 100 -> 1k
- R4: value 10k -> 100
- U1: value DAC7311xDCK -> GAQY212GS; footprint Package_TO_SOT_SMD:SOT-363_SC-70-6 -> Package_SO:SOP-4_3.8x4.1mm_P2.54mm
- U3: value ADuM1300xRW -> LM4040DBZ-5; footprint Package_SO:SOIC-16W_7.5x10.3mm_P1.27mm -> Package_TO_SOT_SMD:SOT-23
- U4: value LM4040DBZ-5 -> ADuM1400xRW; footprint Package_TO_SOT_SMD:SOT-23 -> Package_SO:SOIC-16W_7.5x10.3mm_P1.27mm
- moved U1 52.0 mm to (-7.40, -50.7), turned to 0 degrees
- moved D2 46.1 mm to (90.8, -55.2)
- moved D3 46.1 mm to (90.8, -51.9)
- moved D1 46.1 mm to (90.8, -58.5)
- moved C1 45.3 mm to (99.4, -72.2)
- moved U3 40.0 mm to (93.0, -71.2), turned to 0 degrees
- moved C5 33.8 mm to (68.6, -67.2)
- moved C3 33.8 mm to (68.6, -72.2)
- moved C4 33.8 mm to (68.6, -69.7)
- moved C9 28.5 mm to (68.6, -59.6)
- moved C8 27.8 mm to (68.6, -62.2)
- moved FB2 25.3 mm to (99.4, -69.7)
- moved FB4 25.3 mm to (99.4, -64.7)
- moved FB3 25.3 mm to (99.4, -67.2)
- moved C11 23.9 mm to (90.7, -45.1)
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- renumbered IC27 to IC5, IC28 to IC6, IC29 to IC7, IC30 to IC8
Connections:
- C1 pad 1: Net-(U1-GND) -> Net-(C1-Pad1)
- C1 pad 2: Net-(IC27-VCC) -> Net-(C1-Pad2)
- C10 pad 1: GND -> Net-(U5-V_{DD2})
- C10 pad 2: +3.3V -> Net-(U5-V_{DD2})
- C11 pad 1: +3.3V -> Net-(U6-+Vout)
- C11 pad 2: GND -> Net-(U2-GND)
- C12 pad 1: Net-(U1-GND) -> Net-(U2-GND)
- C12 pad 2: Net-(IC27-VCC) -> Net-(U4-VDD1)
- C2 pad 1: Net-(U1-AVDD/AVREF) -> Net-(C1-Pad2)
- C2 pad 2: Net-(U1-GND) -> Net-(C1-Pad1)
- C3 pad 2: Net-(D33-A2) -> Net-(D1-A2)
- C5 pad 2: Net-(D2-A2) -> Net-(D1-A2)
- C6 pad 2: Net-(D3-A2) -> Net-(D1-A2)
- C7 pad 1: Net-(U1-VOUT) -> Net-(U2-VOUT)
- C7 pad 2: Net-(U1-GND) -> Net-(U2-GND)
- C8 pad 1: Net-(IC27-VCC) -> Net-(U2-AVDD/AVREF)
- C8 pad 2: Net-(U1-GND) -> Net-(U2-GND)
- C9 pad 1: +5V -> Net-(U2-GND)
- C9 pad 2: GND -> Net-(U6-+Vout)
- D2 pad 2: Net-(D2-A2) -> Net-(D1-A2)
- D3 pad 2: Net-(D3-A2) -> Net-(D1-A2)
- FB1 pad 1: Net-(FB1-Pad1) -> -12V
- FB1 pad 2: Net-(IC27-VCC) -> Net-(FB1-Pad2)
- FB2 pad 1: Net-(IC1-VCC+) -> +3.3V
- FB2 pad 2: Net-(IC27-VCC) -> Net-(FB2-Pad2)
- FB3 pad 1: Net-(IC2-VCC+) -> +5V
- FB3 pad 2: Net-(IC27-VCC) -> Net-(FB3-Pad2)
- FB4 pad 1: Net-(IC3-VCC+) -> +12V
- FB4 pad 2: Net-(IC27-VCC) -> Net-(FB4-Pad2)
- FB5 pad 1: Net-(IC4-VCC+) -> Net-(IC1-VCC+)
- FB5 pad 2: Net-(IC27-VCC) -> Net-(U6-+Vout)
- FB6 pad 1: +12V -> Net-(IC2-VCC+)
- FB6 pad 2: Net-(FB6-Pad2) -> Net-(U6-+Vout)
- FB7 pad 1: +5V -> Net-(IC3-VCC+)
- FB7 pad 2: Net-(FB7-Pad2) -> Net-(U6-+Vout)
- FB8 pad 1: +3.3V -> Net-(IC4-VCC+)
- FB8 pad 2: Net-(FB8-Pad2) -> Net-(U6-+Vout)
- FB9 pad 1: -12V -> Net-(FB9-Pad1)
- FB9 pad 2: Net-(FB9-Pad2) -> Net-(U6-+Vout)
- IC1 pad 2: Net-(D33-A2) -> Net-(D1-A2)
- IC3 pad 1: Net-(IC29-A) -> Net-(IC3-OUT)
- IC3 pad 2: Net-(D2-A2) -> Net-(D1-A2)
- IC4 pad 2: Net-(D3-A2) -> Net-(D1-A2)
- IC5 pad 4: Net-(IC27-Y) -> Net-(IC5-Y)
- IC5 pad 5: Net-(IC27-VCC) -> Net-(IC5-VCC)
- IC6 pad 4: Net-(IC28-Y) -> Net-(IC6-Y)
- IC6 pad 5: Net-(IC27-VCC) -> Net-(IC6-VCC)
- IC7 pad 2: Net-(IC29-A) -> Net-(IC3-OUT)
- IC7 pad 4: Net-(IC29-Y) -> Net-(IC7-Y)
- IC7 pad 5: Net-(IC27-VCC) -> Net-(IC7-VCC)
- IC8 pad 4: Net-(IC30-Y) -> Net-(IC8-Y)
- IC8 pad 5: Net-(IC27-VCC) -> Net-(IC8-VCC)
- J1 pad 1: unconnected-(J1-Pin_1-Pad1) -> Net-(J1-Pin_1)
- J1 pad 2: unconnected-(J1-Pin_2-Pad2) -> Net-(J1-Pin_2)
- J1 pad 3: unconnected-(J1-Pin_3-Pad3) -> Net-(J1-Pin_3)
- J1 pad 4: unconnected-(J1-Pin_4-Pad4) -> Net-(J1-Pin_4)
- J1 pad 5: unconnected-(J1-Pin_5-Pad5) -> Net-(D1-A2)
- R1 pad 1: Net-(D33-A1) -> Net-(D1-A1)
- R10 pad 1: Net-(D3-A1) -> Net-(IC2-IN+)
- R10 pad 2: Net-(IC4-IN+) -> Net-(IC2-OUT)
- R11 pad 1: Net-(U1-VOUT) -> Net-(IC3-IN+)
- R11 pad 2: Net-(IC4-IN-) -> Net-(IC3-OUT)
- R13 pad 2: Net-(IC27-Y) -> Net-(IC5-Y)
- R14 pad 2: Net-(IC28-Y) -> Net-(IC6-Y)
- R15 pad 1: Net-(IC29-A) -> Net-(IC3-OUT)
- R15 pad 2: Net-(IC29-Y) -> Net-(IC7-Y)
- R16 pad 2: Net-(IC30-Y) -> Net-(IC8-Y)
- R17 pad 1: Net-(U1-AVDD/AVREF) -> Net-(U2-AVDD/AVREF)
- R17 pad 2: Net-(FB1-Pad1) -> Net-(FB9-Pad1)
- R2 pad 1: Net-(IC1-IN+) -> Net-(U2-VOUT)
- R2 pad 2: Net-(IC1-OUT) -> Net-(IC1-IN-)
- R3 pad 1: Net-(U1-VOUT) -> Net-(D2-A1)
- R3 pad 2: Net-(IC1-IN-) -> Net-(IC2-IN+)
- R4 pad 1: Net-(D1-A1) -> Net-(U2-VOUT)
- R4 pad 2: Net-(IC2-IN+) -> Net-(IC2-IN-)
- R5 pad 1: Net-(U1-VOUT) -> Net-(D3-A1)
- R5 pad 2: Net-(IC2-IN-) -> Net-(IC3-IN+)
- R6 pad 1: Net-(IC2-IN+) -> Net-(U2-VOUT)
- R6 pad 2: Net-(IC2-OUT) -> Net-(IC3-IN-)
- R7 pad 1: Net-(D2-A1) -> Net-(D4-A1)
- R7 pad 2: Net-(IC3-IN+) -> Net-(IC4-IN+)
- R8 pad 1: Net-(U1-VOUT) -> Net-(U2-VOUT)
- R8 pad 2: Net-(IC3-IN-) -> Net-(IC4-IN-)
- R9 pad 1: Net-(IC3-IN+) -> Net-(IC1-IN+)
- R9 pad 2: Net-(IC29-A) -> Net-(IC1-OUT)
- U1 pad 1: Net-(U1-~{SYNC}) -> Net-(R39-Pad2)
- U1 pad 2: Net-(U1-SCLK) -> Net-(R39-Pad1)
- U1 pad 3: Net-(U1-DIN) -> Net-(R20-Pad1)
- U1 pad 4: Net-(U1-AVDD/AVREF) -> Net-(J1-Pin_1)
- U3 pad 1: +3.3V -> Net-(U2-AVDD/AVREF)
- U3 pad 2: GND -> Net-(U2-GND)
- U3 pad 3: /Frontend/MOSI -> unconnected-(U3-NC-Pad3)
- U4 pad 1: Net-(U1-AVDD/AVREF) -> Net-(U4-VDD1)
- U4 pad 2: Net-(U1-GND) -> Net-(U2-GND)
- U4 pad 3: unconnected-(U4-NC-Pad3) -> Net-(IC5-Y)
- X1 pad 1: Net-(FB6-Pad2) -> Net-(FB4-Pad2)
- X1 pad 2: Net-(FB6-Pad2) -> Net-(FB4-Pad2)
- X1 pad 3: Net-(FB7-Pad2) -> Net-(FB3-Pad2)
- X1 pad 4: Net-(FB7-Pad2) -> Net-(FB3-Pad2)
- X1 pad 5: Net-(FB8-Pad2) -> Net-(FB2-Pad2)
- X1 pad 6: Net-(FB8-Pad2) -> Net-(FB2-Pad2)
- X1 pad 7: Net-(FB9-Pad2) -> Net-(FB1-Pad2)
- X1 pad 8: Net-(FB9-Pad2) -> Net-(FB1-Pad2)
Routing:
- net Net-(U1-DIN): track 11.8 -> 0.00 mm
- net Net-(U1-~{SYNC}): track 9.31 -> 0.00 mm
- net Net-(U1-GND): track 8.38 -> 0.00 mm, vias 1 -> 0
- net Net-(U1-SCLK): track 8.27 -> 0.00 mm
- net Net-(U1-AVDD/AVREF): track 5.51 -> 0.00 mm
- net Net-(U1-VOUT): track 1.71 -> 0.00 mm
- net Net-(FB1-Pad1): track 1.57 -> 0.00 mm
- net Net-(IC8-Y): track 0.00 -> 1.18 mm
- net Net-(IC6-Y): track 0.00 -> 1.16 mm
- net Net-(IC5-Y): track 0.00 -> 1.16 mm
- net Net-(IC7-Y): track 0.00 -> 1.15 mm
- net Net-(IC3-OUT): track 0.00 -> 1.11 mm
- net Net-(IC1-OUT): track 0.00 -> 1.10 mm
- net Net-(IC2-OUT): track 0.00 -> 1.09 mm
- net Net-(IC4-OUT): track 0.00 -> 1.08 mm
