File: pcb/TSC_board.kicad_pcb (KiCad board)
At the start: 4 copper layers, 100 x 100 mm, 390 parts, among them IC1 TS3021ILT, IC10 TS3021ILT, IC11 TS3021ILT, IC12 TS3021ILT, IC13 TS3021ILT, IC14 TS3021ILT, IC2 TS3021ILT, IC3 TS3021ILT, IC4 TS3021ILT, IC5 TS3021ILT, IC6 TS3021ILT, IC7 TS3021ILT, IC8 TS3021ILT, IC9 TS3021ILT, J1 Conn_01x05_Socket, J2 Conn_01x05_Socket, J3 Conn_01x04_Socket, J4 Conn_01x04_Socket, U1 TEA1-0505, U10 ADuM1400xRW, U11 GAQY212GS, U12 GAQY212GS, U13 GAQY212GS, U14 GAQY212GS, U15 LM4040DBZ-5, U16 DAC7311xDCK, U17 ADuM1300xRW, U18 TEA1-0505, U19 GAQY212GS, U2 GAQY212GS, U20 GAQY212GS, U21 GAQY212GS, U22 GAQY212GS, U23 GAQY212GS, U24 GAQY212GS, U25 GAQY212GS, U26 GAQY212GS, U27 ADuM1400xRW, U28 GAQY212GS, U29 GAQY212GS, U3 GAQY212GS, U30 GAQY212GS, U31 GAQY212GS, U32 LM4040DBZ-5, U33 DAC7311xDCK, U34 ADuM1300xRW, U35 TEA1-0505, U36 GAQY212GS, U37 GAQY212GS, U38 GAQY212GS, U39 GAQY212GS, U4 GAQY212GS, U40 GAQY212GS, U41 GAQY212GS, U42 ADuM1300xRW, U43 GAQY212GS, U44 GAQY212GS, U45 GAQY212GS, U46 LM4040DBZ-5, U47 DAC7311xDCK, U48 ADuM1300xRW, U49 TEA1-0505, U5 GAQY212GS, U50 GAQY212GS, U51 GAQY212GS, U52 GAQY212GS, U53 GAQY212GS, U54 GAQY212GS, U55 GAQY212GS, U56 ADuM1300xRW, U57 GAQY212GS, U58 GAQY212GS, U59 GAQY212GS, U6 GAQY212GS, U60 LM4040DBZ-5, U61 DAC7311xDCK, U62 ADuM1300xRW, U63 APS6404L-3SQRx-SN, U7 GAQY212GS, U8 GAQY212GS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

Commit message: Update schematic, more routing
Add firmware/TSC_RangeControl.ioc (STM32CubeMX project for STM32C011F4Px). Numerous adjustments to the schematic. Update PCB files.
Parts:
- C19, C20, C3, C35, C36, C4, C50, C51, R107, R158, R167, R182, R58, R69, R88: moved to B.Cu
- moved R118 259.7 mm to (123.7, 163.9)
- moved R119 259.7 mm to (123.7, 166.4)
- moved R122 259.7 mm to (123.7, 173.9)
- moved R125 259.7 mm to (123.7, 181.4)
- moved R126 259.7 mm to (123.7, 183.9)
- moved R131 259.7 mm to (123.7, 196.5)
- moved R134 259.7 mm to (123.7, 204.0)
- moved R135 259.7 mm to (123.7, 206.5)
- moved R137 259.7 mm to (127.7, 156.3)
- moved R138 259.7 mm to (127.7, 158.8)
- moved R140 259.7 mm to (127.7, 163.9)
- moved R141 259.7 mm to (127.7, 166.4)
- moved R144 259.7 mm to (127.7, 173.9)
- moved R147 259.7 mm to (127.7, 181.4)
- moved R148 259.7 mm to (127.7, 183.9)
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Connections:
- C12 pad 2: Net-(U17-V_{DD2}) -> Net-(D1-A2)
- C28 pad 2: Net-(U34-V_{DD2}) -> Net-(D5-A2)
- C58 pad 2: Net-(U62-V_{DD2}) -> Net-(D12-A2)
Routing:
- net Net-(U16-VOUT): track 0.00 -> 41.0 mm, vias 0 -> 5
- net Net-(U1-+Vout): track 0.00 -> 39.5 mm, vias 0 -> 1
- net Net-(U18-+Vout): track 0.00 -> 39.4 mm, vias 0 -> 1
- net Net-(U61-VOUT): track 0.00 -> 37.0 mm, vias 0 -> 4
- net Net-(U33-VOUT): track 0.00 -> 33.9 mm, vias 0 -> 4
- net Net-(U49-+Vout): track 0.00 -> 33.7 mm, vias 0 -> 1
- net Net-(IC8-OUT): track 0.00 -> 28.9 mm, vias 0 -> 2
- net Net-(IC14-OUT): track 0.00 -> 26.3 mm, vias 0 -> 2
- net Net-(IC7-OUT): track 0.00 -> 25.3 mm, vias 0 -> 2
- net Net-(IC6-OUT): track 0.00 -> 23.8 mm, vias 0 -> 2
- net Net-(IC13-OUT): track 0.00 -> 23.7 mm, vias 0 -> 2
- net Net-(IC5-OUT): track 0.00 -> 23.3 mm, vias 0 -> 2
- net Net-(IC12-OUT): track 0.00 -> 23.1 mm, vias 0 -> 2
- net Net-(D5-A2): track 0.00 -> 22.0 mm, vias 0 -> 5
- net Net-(D12-A2): track 0.00 -> 18.5 mm, vias 0 -> 4
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- added copper zone on B.Cu, net Net-(D12-A2)
- added copper zone on F.Cu, net Net-(D12-A2)
- added copper zone on In1.Cu, net Net-(D12-A2)
- added copper zone on In2.Cu, net Net-(D12-A2)
- added copper zone on B.Cu, net Net-(D5-A2)
- added copper zone on F.Cu, net Net-(D5-A2)
- added copper zone on In1.Cu, net Net-(D5-A2)
- added copper zone on In2.Cu, net Net-(D5-A2)
