File: pcb/Frontend.kicad_sch (KiCad schematic)
At the start: 39 parts, among them IC27 NL17SZ17DFT2G, IC28 NL17SZ17DFT2G, IC29 NL17SZ17DFT2G, IC30 NL17SZ17DFT2G, IC31 NL17SZ17DFT2G, IC32 NL17SZ17DFT2G, IC33 NL17SZ17DFT2G, IC34 NL17SZ17DFT2G, IC35 NL17SZ17DFT2G, IC36 NL17SZ17DFT2G, IC37 NL17SZ17DFT2G, IC38 NL17SZ17DFT2G, IC39 NL17SZ17DFT2G, IC40 NL17SZ17DFT2G, U27 ADuM1300xRW, U28 ADuM1300xRW, U29 TEA1-0505, U30 TEA1-0505, U31 TEA1-0505, U32 TEA1-0505, U7 ADuM1400xRW, U8 ADuM1400xRW

Commit message: Change of concept, only frontend. To be connected with UCB_board
Parts:
- removed C65: 10n, Capacitor_SMD:C_0603_1608Metric_Pad1.08x0.95mm_HandSolder, symbol Device:C
- added C1, C11, C2, C3, C4, C5, C6: 100n, Capacitor_SMD:C_0603_1608Metric_Pad1.08x0.95mm_HandSolder, symbol Device:C
- added C10: 10n, Capacitor_SMD:C_0603_1608Metric_Pad1.08x0.95mm_HandSolder, symbol Device:C
- added C7: 1n, Capacitor_SMD:C_0603_1608Metric_Pad1.08x0.95mm_HandSolder, symbol Device:C
- added C8, C9: 10u, Capacitor_SMD:C_1206_3216Metric, symbol Device:C
- added D1, D2, D3: SMF5.0CA, Diode_SMD:D_SMF, symbol Diode:SMF5V0A
- added IC1, IC2, IC3, IC4: TS3021ILT, SOT95P280X145-5N, symbol TS3021ILT:TS3021ILT
- added R1, R10, R4, R7: 10k, Resistor_SMD:R_0603_1608Metric, symbol Device:R
- added R11, R3, R5, R8: 100, Resistor_SMD:R_0603_1608Metric, symbol Device:R
- added R12, R2, R6, R9: 100k, Resistor_SMD:R_0603_1608Metric, symbol Device:R
- added R13, R14, R15, R16: 0R, Resistor_SMD:R_0402_1005Metric, symbol Device:R
- added R17: (no value), Resistor_SMD:R_0603_1608Metric, symbol Device:R
- added U1: DAC7311xDCK, Package_TO_SOT_SMD:SOT-363_SC-70-6, symbol Analog_DAC:DAC7311xDCK
- added U3: ADuM1300xRW, Package_SO:SOIC-16W_7.5x10.3mm_P1.27mm, symbol Isolator:ADuM1300xRW
- added U4: LM4040DBZ-5, Package_TO_SOT_SMD:SOT-23, symbol Reference_Voltage:LM4040DBZ-5
- IC27, IC28, IC29, IC30: now not fitted; now left out of the parts list
Connections:
- net +3.3V: now also C10.2, C11.1, U3.1 (V_{DD1})
- net +5V: now also C9.1
- net GND: now also C10.1, C11.2, C9.2, U3.2 (GND_{1}), U3.8 (GND_{1})
- net at IC27.3 (GND), IC28.3 (GND), IC29.3 (GND)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: now also C1.1, C2.2, C7.2, C8.2, U1.5 (GND), U3.15 (GND_{2}), U3.9 (GND_{2}), U4.2 (A)
- net at IC27.5 (VCC), IC28.5 (VCC), IC29.5 (VCC)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: now also C1.2, C8.1, R17.2, U3.10 (V_{E2}), U3.16 (V_{DD2})
- net at D33.1 (A1): now also R1.1
- net at D33.2 (A2): now also C3.2, IC1.2 (VCC-)
- net at IC29.2 (A): now also IC3.1 (OUT), R15.1, R9.2
- net at IC29.4 (Y), U8.5 (VIC): now also R15.2
- net at IC28.2 (A): now also IC2.1 (OUT), R14.1, R6.2
- net at IC28.4 (Y), U8.4 (VIB): now also R14.2
- net at IC27.2 (A): now also IC1.1 (OUT), R13.1, R2.2
- net at IC27.4 (Y), U8.3 (VIA): now also R13.2
- net at IC30.2 (A): now also IC4.1 (OUT), R12.2, R16.1
- net at IC30.4 (Y), U8.6 (VID): now also R16.2
- new net: C3.1, IC1.5 (VCC+)
- new net: D2.1 (A1), R7.1
- new net: IC3.3 (IN+), R7.2, R9.1
- new net: U1.1 (~{SYNC}), U3.12 (V_{OC})
- new net: U1.2 (SCLK), U3.13 (V_{OB})
- new net: U1.3 (DIN), U3.14 (V_{OA})
- new net: C2.1, R17.1, U1.4 (AVDD/AVREF), U4.1 (K)
- new net: C7.1, R11.1, R3.1, R5.1, R8.1, U1.6 (VOUT)
- new net: IC3.4 (IN-), R8.2
- new net: C5.2, D2.2 (A2), IC3.2 (VCC-)
- new net: C5.1, IC3.5 (VCC+)
- new net: D3.1 (A1), R10.1
- new net: IC4.3 (IN+), R10.2, R12.1
- new net: IC4.4 (IN-), R11.2
- new net: IC1.3 (IN+), R1.2, R2.1
- new net: IC1.4 (IN-), R3.2
- new net: D1.1 (A1), R4.1
- new net: IC2.3 (IN+), R4.2, R6.1
- new net: C6.2, D3.2 (A2), IC4.2 (VCC-)
- new net: C6.1, IC4.5 (VCC+)
- new net: C4.2, D1.2 (A2), IC2.2 (VCC-)
- new net: IC2.4 (IN-), R5.2
- new net: C4.1, IC2.5 (VCC+)
- new net CS1: U3.5 (V_{IC})
- new net MOSI: U3.3 (V_{IA})
- new net SCK: U3.4 (V_{IB})
Other:
- moved on the sheet: C56, C57, C58, C59, C60, C61, C62, C63, C64, C66, C67, C68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

Commit message: Add STM32 .ioc and adjust UCB connector footprint
Add STM32CubeMX project file (firmware/TSC_board.ioc) for the STM32H563VITx MCU and update KiCad PCB/schematic files. Adjust UCB_conn footprint and apply corresponding changes to pcb TSC_board/Frontend/MCU schematic and project files to reflect the connector/placement updates.
Parts:
- added C12: 100n, Capacitor_SMD:C_0603_1608Metric, symbol Device:C
- added FB1, FB2, FB3, FB4, FB5: 100R @ 100MHz, Inductor_SMD:L_0603_1608Metric, symbol Device:FerriteBead_Small
- added J1, J2: Conn_01x05_Socket, Connector_Phoenix_MC:PhoenixContact_MC_1,5_5-G-3.5_1x05_P3.50mm_Horizontal, symbol Connector:Conn_01x05_Socket
- added J3, J4: Conn_01x04_Socket, Connector_Phoenix_MC:PhoenixContact_MC_1,5_4-G-3.5_1x04_P3.50mm_Horizontal, symbol Connector:Conn_01x04_Socket
- added U2: CPC1006N, Package_SO:SOP-4_3.8x4.1mm_P2.54mm, symbol Relay_SolidState:CPC1006N
- C1, C10, C11, C2, C3, C4, C5, C6, C67, C69, C7, C71: footprint Capacitor_SMD:C_0603_1608Metric_Pad1.08x0.95mm_HandSolder -> Capacitor_SMD:C_0603_1608Metric
- C56, C57, C58, C59, C60, C61, C62, C63, C64, C66, C68, C70, IC31, IC32, IC33, IC34, IC35, IC36, IC37, IC38, IC39, IC40, U27, U28, U30, U31, U32, U7: now not fitted; now left out of the parts list
- R17: value (none) -> 330R
Connections:
- net at C3.1, IC1.5 (VCC+): now also FB2.1
- net at C1.1, C2.2, C7.2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: now also C12.1; no longer IC27.3 (GND), IC28.3 (GND), IC29.3 (GND), IC30.3 (GND)
- net at C1.2, C8.1, IC27.5 (VCC)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: now also C12.2, FB1.2, FB2.2, FB3.2, FB4.2, FB5.2; no longer R17.2
- net at C5.1, IC3.5 (VCC+): now also FB4.1
- net at C6.1, IC4.5 (VCC+): now also FB5.1
- net at C4.1, IC2.5 (VCC+): now also FB3.1
- new net: IC27.3 (GND), IC28.3 (GND), IC29.3 (GND), IC30.3 (GND)
- new net: FB1.1, R17.2
Other:
- moved on the sheet: C10, C11, C2, C7, IC27, IC28, IC29, IC30, R13, R14, R15, R16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

Commit message: More schematic
Parts:
- removed U2: CPC1006N, Package_SO:SOP-4_3.8x4.1mm_P2.54mm, symbol Relay_SolidState:CPC1006N
- added C10, C31, C32, C33, C34: 100n, Capacitor_SMD:C_0603_1608Metric, symbol Device:C
- added FB10, FB11, FB12, FB13, FB14, FB15: 100R @ 100MHz, Inductor_SMD:L_0603_1608Metric, symbol Device:FerriteBead_Small
- added R18, R19, R20, R21, R22, R23, R24, R25, R26, R27, R28, R29, R30, R31, R32, R33, R34, R35, R36, R37, R38, R39, R40, R41, R42, R43, R44, R45, R46, R47, R48, R49: 10k, Resistor_SMD:R_0603_1608Metric, symbol Device:R
- added R50, R51, R52, R53, R54, R55, R56, R57, R58, R59, R60, R61: 470, Resistor_SMD:R_0603_1608Metric, symbol Device:R
- added U1, U13, U14, U15, U16, U17, U18, U19, U21, U22, U23, U24: GAQY212GS, Package_SO:SOP-4_3.8x4.1mm_P2.54mm, symbol Relay_SolidState:CPC1006N
- IC1, IC2, IC3, IC4: footprint SOT95P280X145-5N -> TS3021ILT:SOT95P280X145-5N
- R1: value 10k -> 1k
- R10: renamed from R6; value 100k -> 50k
- R11: renamed from R9; value 100k -> 50k
- R12: value 100k -> 50k
- R3: renamed from R4; value 10k -> 1k
- R5: renamed from R7; value 10k -> 1k
- R7: renamed from R10; value 10k -> 1k
- R9: renamed from R2; value 100k -> 50k
- renumbered C8 to C11, C9 to C13, C69 to C14, C64 to C15, C56 to C16, C60 to C17, C67 to C18, C71 to C19, C10 to C20, C66 to C21, C57 to C22, C61 to C23, C68 to C24, C11 to C25, C58 to C26, C62 to C27, C70 to C28, C59 to C29, C63 to C30, C2 to C8, C1 to C9, D33 to D1, D1 to D2, D2 to D3, D3 to D4, FB2 to FB5, FB3 to FB6, FB4 to FB7, FB5 to FB8, FB1 to FB9, IC32 to IC10, IC33 to IC11, IC34 to IC12, IC35 to IC13, IC36 to IC14, IC37 to IC15, IC38 to IC16, IC39 to IC17, IC40 to IC18, IC27 to IC5, IC28 to IC6, IC29 to IC7, IC30 to IC8, IC31 to IC9, R3 to R2, R5 to R4, R8 to R6, R11 to R8, U7 to U10, U28 to U11, U27 to U12, U1 to U2, U4 to U3, U8 to U4, U3 to U5, U29 to U6, U30 to U7, U31 to U8, U32 to U9
Connections:
- net +5V: now also R50.1, R51.1, R52.1, R53.1, R54.1, R55.1, R56.1, R57.1, R58.1, R59.1, R60.1, R61.1
- net at C3.2, D1.2 (A2), IC1.2 (VCC-): now also C4.2, C5.2, C6.2, D2.2 (A2), D3.2 (A2), D4.2 (A2), IC2.2 (VCC-), IC3.2 (VCC-), IC4.2 (VCC-), J1.5 (Pin_5), R18.2, R27.2, R32.2, R37.2
- net at C11.1, C9.2, FB5.2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: now also FB10.2, FB11.2, FB12.2, FB13.2, FB14.2, FB15.2; no longer C12.2, IC5.5 (VCC), IC6.5 (VCC), IC7.5 (VCC), IC8.5 (VCC), U4.1 (VDD1), U5.10 (V_{E2}), U5.16 (V_{DD2})
- net at D3.1 (A1), R5.1: now also R31.2, R32.1, U21.3
- net at D4.1 (A1), R7.1: now also R36.2, R37.1, U24.3
- net at D1.1 (A1), R1.1: now also R18.1, R19.2, U14.3
- net at D2.1 (A1), R3.1: now also R26.2, R27.1, U17.3
- net at IC5.3 (GND), IC6.3 (GND), IC7.3 (GND)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: now also C31.2, C32.2, C33.2, C34.2
- net at J1.1 (Pin_1): now also U1.4, U13.4, U14.4
- net at J1.2 (Pin_2): now also U15.4, U16.4, U17.4
- net at J1.3 (Pin_3): now also U18.4, U19.4, U21.4
- net at J1.4 (Pin_4): now also U22.4, U23.4, U24.4
- new net: R41.2, R54.2, U15.1
- new net: C32.1, FB13.1, IC6.5 (VCC)
- new net: R46.1, U18.2
- new net: R46.2, R57.2, U18.1
- new net: R44.2, R58.2, U21.1
- new net: C10.1, C10.2, FB11.1, U5.10 (V_{E2}), U5.16 (V_{DD2})
- new net: R43.2, R55.2, U17.1
- new net: R28.2, R29.1
- new net: R29.2, R30.1, U19.3
- new net: R47.2, R61.2, U24.1
- new net: R47.1, U24.2
- new net: R20.1, R21.2, U1.3
- new net: R19.1, R20.2
- new net: C31.1, FB12.1, IC5.5 (VCC)
- new net: R49.2, R60.2, U22.1
- new net: R49.1, U22.2
- new net: R33.1, U22.3
- new net: R42.2, R53.2, U16.1
- new net: R42.1, U16.2
- new net: R24.2, R25.1, U16.3
- new net: C33.1, FB14.1, IC7.5 (VCC)
- new net: R38.2, R50.2, U13.1
- new net: R38.1, U13.2
- new net: R22.1, U13.3
- new net: R48.2, R59.2, U23.1
- new net: R48.1, U23.2
- new net: R34.2, R35.1, U23.3
- new net: R41.1, U15.2
- new net: R23.1, U15.3
- new net: R33.2, R34.1
- new net: C34.1, FB15.1, IC8.5 (VCC)
- new net: R39.2, R51.2, U1.1
- new net: R39.1, U1.2
- new net: R35.2, R36.1
- new net: R23.2, R24.1
- new net: R43.1, U17.2
- new net: R30.2, R31.1
- new net: R45.1, U19.2
- new net: R45.2, R56.2, U19.1
- new net: R40.2, R52.2, U14.1
- new net: R40.1, U14.2
- new net: R21.1, R22.2
- new net: R25.2, R26.1
- new net: C12.2, FB10.1, U4.1 (VDD1)
- new net: R28.1, U18.3
- new net: R44.1, U21.2
Other:
- moved on the sheet: C12, J1, J2, J3, J4

Commit message: Remove NL17SZ17 symbol; update schematic
Delete the NL17SZ17DFT2G symbol from pcb/Frontend.kicad_sch and apply a bulk update to schematic. Many junction coordinates and UUIDs were regenerated/adjusted in Frontend.kicad_sch; related KiCad files (pcb/MCU.kicad_sch, pcb/TSC_board.kicad_pcb, pcb/TSC_board.kicad_sch) were also updated. This is primarily a cleanup refresh.
Parts:
- removed C13: 10u, Capacitor_SMD:C_1206_3216Metric, symbol Device:C
- removed C15, C16: 10n, Capacitor_SMD:C_0603_1608Metric_Pad1.08x0.95mm_HandSolder, symbol Device:C
- removed IC10, IC11, IC12, IC13, IC14, IC15, IC16, IC17, IC18, IC5, IC6, IC7, IC8, IC9: NL17SZ17DFT2G, SOT65P210X110-5N, symbol SamacSys_Parts:NL17SZ17DFT2G
- removed R13, R14, R15, R16: 0R, Resistor_SMD:R_0402_1005Metric, symbol Device:R
- removed U10: ADuM1400xRW, Package_SO:SOIC-16W_7.5x10.3mm_P1.27mm, symbol Isolator:ADuM1400xRW
- removed U11, U12: ADuM1300xRW, Package_SO:SOIC-16W_7.5x10.3mm_P1.27mm, symbol Isolator:ADuM1300xRW
- removed U7, U8, U9: TEA1-0505, Converter_DCDC:Converter_DCDC_TRACO_TEA1-xxxx_THT, symbol Converter_DCDC:TEA1-0505
- added C18, C49: 10u, Capacitor_SMD:C_1206_3216Metric, symbol Device:C
- added C19, C3, C35, C39, C45, C50, C54, C60: 10n, Capacitor_SMD:C_0603_1608Metric, symbol Device:C
- added C20, C25, C36, C37, C38, C40, C41, C42, C43, C44, C46, C48, C51, C52, C53, C55, C56, C57, C58, C59, C61: 100n, Capacitor_SMD:C_0603_1608Metric, symbol Device:C
- added C47, C62: 1n, Capacitor_SMD:C_0603_1608Metric, symbol Device:C
- added D10, D11, D12, D13, D14, D5, D6, D7, D8, D9: SMF5.0CA, Diode_SMD:D_SMF, symbol Diode:SMF5V0A
- added FB16, FB17, FB18, FB19, FB20, FB21, FB22, FB23, FB24, FB25, FB26, FB27, FB28, FB29, FB30: 100R @ 100MHz, Inductor_SMD:L_0603_1608Metric, symbol Device:FerriteBead_Small
- added IC10, IC11, IC12, IC13, IC14, IC5, IC6, IC7, IC8, IC9: TS3021ILT, TS3021ILT:SOT95P280X145-5N, symbol TS3021ILT:TS3021ILT
- added R100, R101, R103, R104, R105, R106, R110, R111, R112, R113, R121, R122, R123, R125, R126, R127, R133, R134, R135, R136, R137, R138, R140, R141, R142, R147, R148, R149, R151, R152, R153, R154, R155, R156, R164, R165, R166, R168, R169, R170, R176, R177, R178, R179, R180, R181, R183, R184, R185, R190, R191, R192, R194, R195, R196, R197, R198, R199, R65, R66, R67, R68, R70, R71, R72, R73, R80, R81, R82, R83, R84, R85, R86, R87, R89, R90, R91, R92, R98, R99: 10k, Resistor_SMD:R_0603_1608Metric, symbol Device:R
- added R102, R109, R117, R129, R150, R160, R172, R193, R60, R75: 100, Resistor_SMD:R_0603_1608Metric, symbol Device:R
- added R107, R115, R124, R139, R158, R167, R182, R58, R69, R88: 50k, Resistor_SMD:R_0603_1608Metric, symbol Device:R
- added R108, R116, R128, R145, R159, R171, R188, R59, R74, R96: 1k, Resistor_SMD:R_0603_1608Metric, symbol Device:R
- added R114, R157, R200: 330R, Resistor_SMD:R_0603_1608Metric, symbol Device:R
- added R118, R119, R120, R130, R131, R132, R143, R144, R146, R161, R162, R163, R173, R174, R175, R186, R187, R189, R61, R62, R63, R64, R76, R77, R78, R79, R93, R94, R95, R97: 470, Resistor_SMD:R_0603_1608Metric, symbol Device:R
- added U18, U35, U49: TEA1-0505, Converter_DCDC:Converter_DCDC_TRACO_TEA1-xxxx_THT, symbol Converter_DCDC:TEA1-0505
- added U19, U20, U21, U22, U23, U24, U25, U26, U28, U29, U30, U31, U36, U37, U38, U39, U40, U41, U43, U44, U45, U50, U51, U52, U53, U54, U55, U57, U58, U59: GAQY212GS, Package_SO:SOP-4_3.8x4.1mm_P2.54mm, symbol Relay_SolidState:CPC1006N
- added U27: ADuM1400xRW, Package_SO:SOIC-16W_7.5x10.3mm_P1.27mm, symbol Isolator:ADuM1400xRW
- added U32, U46, U60: LM4040DBZ-5, Package_TO_SOT_SMD:SOT-23, symbol Reference_Voltage:LM4040DBZ-5
- added U33, U47, U61: DAC7311xDCK, Package_TO_SOT_SMD:SOT-363_SC-70-6, symbol Analog_DAC:DAC7311xDCK
- added U34, U42, U48, U56, U62: ADuM1300xRW, Package_SO:SOIC-16W_7.5x10.3mm_P1.27mm, symbol Isolator:ADuM1300xRW
- C17, C24, C26, C27: value 10n -> 100n; footprint Capacitor_SMD:C_0603_1608Metric_Pad1.08x0.95mm_HandSolder -> Capacitor_SMD:C_0603_1608Metric; now fitted; now in the parts list
- C21, C22, C28, C29: footprint Capacitor_SMD:C_0603_1608Metric_Pad1.08x0.95mm_HandSolder -> Capacitor_SMD:C_0603_1608Metric; now fitted; now in the parts list
- C23, C30: value 100n -> 10n; footprint Capacitor_SMD:C_0603_1608Metric_Pad1.08x0.95mm_HandSolder -> Capacitor_SMD:C_0603_1608Metric; now fitted; now in the parts list
- C31, C33, FB12, FB13, FB14, FB15: now fitted; now in the parts list
- C32: value 100n -> 1n; now fitted; now in the parts list
- C34: value 100n -> 10u; footprint Capacitor_SMD:C_0603_1608Metric -> Capacitor_SMD:C_1206_3216Metric; now fitted; now in the parts list
- renumbered C9 to C1, C5 to C10, C6 to C11, C10 to C12, C8 to C13, C20 to C14, C25 to C15, C7 to C16, C11 to C2, C18 to C4, C3 to C5, C12 to C6, C14 to C7, C19 to C8, C4 to C9, FB11 to FB10, FB9 to FB11, FB10 to FB6, FB6 to FB7, FB7 to FB8, FB8 to FB9, R9 to R1, R46 to R10, R49 to R11, R10 to R12, R22 to R13, R23 to R14, R28 to R15, R33 to R16, R3 to R17, R4 to R18, R51 to R19, R1 to R2, R53 to R20, R56 to R21, R59 to R22, R21 to R23, R29 to R25, R34 to R26, R39 to R27, R42 to R28, R45 to R29, R2 to R3, R48 to R30, R11 to R31, R20 to R32, R25 to R33, R30 to R34, R55 to R36, R58 to R37, R61 to R38, R5 to R39, R50 to R4, R52 to R40, R19 to R41, R26 to R42, R31 to R43, R36 to R44, R6 to R45, R43 to R46, R44 to R47, R47 to R48, R40 to R49, R54 to R5, R12 to R50, R7 to R51, R8 to R52, R18 to R53, R27 to R54, R32 to R55, R37 to R56, R17 to R57, R57 to R6, R60 to R7, R38 to R8, R41 to R9, U6 to U1, U4 to U10, U17 to U11, U21 to U12, U24 to U13, U3 to U15, U2 to U16, U5 to U17, U13 to U2, U15 to U3, U18 to U4, U22 to U5, U1 to U6, U16 to U7, U19 to U8, U23 to U9
Connections:
- net +3.3V: now also C23.2, C24.1, C30.2, C31.1, C39.2, C40.1, C45.2, C46.1, C54.2, C55.1, C60.2, C61.1, U27.10 (VE2), U27.16 (VDD2), U34.1 (V_{DD1}), U42.10 (V_{E2}), U42.16 (V_{DD2}), U48.1 (V_{DD1}), U56.10 (V_{E2}), U56.16 (V_{DD2}), U62.1 (V_{DD1}); no longer C24.2, C26.2, C27.2, C28.1, C29.1, C30.1
- net +5V: now also C19.2, C20.1, C3.2, C35.2, C36.1, C50.2, C51.1, R118.1, R119.1, R120.1, R130.1, R131.1, R132.1, R143.1, R144.1, R146.1, R161.1, R162.1, R163.1, R173.1, R174.1, R175.1, R186.1, R187.1, R189.1, R61.1, R62.1, R63.1, R64.1, R76.1, R77.1, R78.1, R79.1, R93.1, R94.1, R95.1, R97.1, U18.2 (+Vin), U35.2 (+Vin), U49.2 (+Vin); no longer C17.2, C21.1, C22.1, C23.1
- net CH2_1_IN: now also U27.14 (VOA)
- net CH2_2_IN: now also U27.13 (VOB)
- net CH2_3_IN: now also U27.12 (VOC)
- net CH2_4_IN: now also U27.11 (VOD)
- net CH3_1_IN: now also U42.14 (V_{OA})
- net CH3_2_IN: now also U42.13 (V_{OB})
- net CH3_3_IN: now also U42.12 (V_{OC})
- net CH4_1_IN: now also U56.14 (V_{OA})
- net CH4_2_IN: now also U56.13 (V_{OB})
- net CH4_3_IN: now also U56.12 (V_{OC})
- net GND: now also C23.1, C24.2, C30.1, C31.2, C19.1, C20.2, C3.1, C35.1, C36.2, C39.1, C40.2, C45.1, C46.2, C50.1, C51.2, C54.1, C55.2, C60.1, C61.2, U18.1 (-Vin), U27.15 (GND2), U27.9 (GND2), U34.2 (GND_{1}), U34.8 (GND_{1}), U35.1 (-Vin), U42.15 (GND_{2}), U42.9 (GND_{2}), U48.2 (GND_{1}), U48.8 (GND_{1}), U49.1 (-Vin), U56.15 (GND_{2}), U56.9 (GND_{2}), U62.2 (GND_{1}), U62.8 (GND_{1}); no longer C17.1, C21.2, C22.2, C23.2, C24.1, C26.1, C27.1, C28.2, C29.2, C30.2
- net at C1.2, C2.1, FB10.2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: no longer FB12.2, FB13.2, FB14.2, FB15.2
- net at C32.1: now also R102.1, R109.1, R60.1, R75.1, U33.6 (VOUT); no longer FB13.1
- net CH1_IN3_R25: now reaches R10.1, U4.2
- net CH1_IN4_R5: now reaches R48.1, U13.2
- net at IC1.1 (OUT), R1.2: now also U10.3 (VIA)
- net at IC3.1 (OUT), R31.2: now also U10.5 (VIC)
- net at FB12.1: now also C21.1, IC5.5 (VCC+); no longer C31.1
- net CH1_IN4_R25: now reaches R11.1, U5.2
- net at IC2.1 (OUT), R12.2: now also U10.4 (VIB)
- net CH1_IN2_R15: now reaches R28.1, U7.2
- net at J3.1 (Pin_1): now also U36.4, U39.4, U45.4
- net at J3.2 (Pin_2): now also U37.4, U40.4, U43.4
- net at J3.3 (Pin_3): now also U38.4, U41.4, U44.4
- net at J3.4 (Pin_4): now also R154.2, R155.2, R156.2
- net at C33.1: now also C34.2, C38.1, C44.2, C47.2, U35.3 (-Vout), U42.2 (GND_{1}), U42.8 (GND_{1}), U46.2 (A), U47.5 (GND), U48.15 (GND_{2}), U48.9 (GND_{2}); no longer FB14.1
- net CH1_IN1_R25: now reaches R8.1, U2.2
- net CH1_IN4_R15: now reaches R30.1, U9.2
- net CH1_IN2_R25: now reaches R9.1, U3.2
- net at C34.1: now also C33.2, FB19.2, FB20.2, FB21.2, FB22.2, FB23.2, FB24.2, U35.4 (+Vout); no longer FB15.1
- net at IC4.1 (OUT), R50.2: now also U10.6 (VID)
- net CH1_IN1_R15: now reaches R27.1, U6.2
- net CH1_IN2_R5: now reaches R46.1, U11.2
- net CH1_IN3_R15: now reaches R29.1, U8.2
- net CH1_IN1_R5: now reaches R49.1, U14.2
- net at J2.1 (Pin_1): now also U19.4, U23.4, U31.4
- net at J2.2 (Pin_2): now also U20.4, U24.4, U28.4
- net at J2.3 (Pin_3): now also U21.4, U25.4, U29.4
- net at J2.4 (Pin_4): now also U22.4, U26.4, U30.4
- net at J2.5 (Pin_5): now also C21.2, C26.2, C27.2, C25.2, D5.2 (A2), D6.2 (A2), D7.2 (A2), D8.2 (A2), IC5.2 (VCC-), IC6.2 (VCC-), IC7.2 (VCC-), IC8.2 (VCC-), R110.2, R111.2, R112.2, R113.2
- net CH1_IN3_R5: now reaches R47.1, U12.2
- net at J4.1 (Pin_1): now also U50.4, U53.4, U59.4
- net at J4.2 (Pin_2): now also U51.4, U54.4, U57.4
- net at J4.3 (Pin_3): now also U52.4, U55.4, U58.4
- net at J4.4 (Pin_4): now also R197.2, R198.2, R199.2
- net CS1 renamed DAC_CS1
- net MOSI renamed DAC_MOSI
- net DAC_MOSI: now also U34.3 (V_{IA}), U48.3 (V_{IA}), U62.3 (V_{IA})
- net SCK renamed DAC_SCK
- net DAC_SCK: now also U34.4 (V_{IB}), U48.4 (V_{IB}), U62.4 (V_{IB})
- new net: R119.2, R122.2, U37.1
- new net: R120.2, R123.2, U38.1
- new net: C53.2, FB26.1, U56.1 (V_{DD1})
- new net: C48.1, C49.2, C53.1, C59.2, C62.2, U49.3 (-Vout), U56.2 (GND_{1}), U56.8 (GND_{1}), U60.2 (A), U61.5 (GND), U62.15 (GND_{2}), U62.9 (GND_{2})
- new net: IC12.1 (OUT), R158.2, U56.3 (V_{IA})
- new net: IC13.1 (OUT), R167.2, U56.4 (V_{IB})
- new net: IC14.1 (OUT), R182.2, U56.5 (V_{IC})
- new net: IC5.3 (IN+), R58.1, R59.2
- new net: IC5.1 (OUT), R58.2, U27.3 (VIA)
- new net: C17.1, C18.2, C22.1, C29.2, C32.2, U18.3 (-Vout), U27.2 (GND1), U27.8 (GND1), U32.2 (A), U33.5 (GND), U34.15 (GND_{2}), U34.9 (GND_{2})
- new net: C17.2, C18.1, FB12.2, FB13.2, FB14.2, FB15.2, FB16.2, FB17.2, FB18.2, U18.4 (+Vout)
- new net: R132.2, R138.2, U41.1
- new net: R135.2, R142.1, U41.3
- new net: D14.1 (A1), R188.1, R192.2, R199.1, U58.3
- new net: C52.2, C56.2, C57.2, D12.2 (A2), D13.2 (A2), D14.2 (A2), IC12.2 (VCC-), IC13.2 (VCC-), IC14.2 (VCC-)
- new net: C56.1, FB27.1, IC13.5 (VCC+)
- new net: FB24.1, R157.2
- new net: D8.1 (A1), R101.2, R108.1, R113.1, U30.3
- new net: R162.2, R165.2, U51.1
- new net: R169.1, U51.3
- new net: R76.2, R84.2, U23.1
- new net: D9.1 (A1), R116.1, R147.2, R154.1, U45.3
- new net: C37.2, C41.2, C42.2, D10.2 (A2), D11.2 (A2), D9.2 (A2), IC10.2 (VCC-), IC11.2 (VCC-), IC9.2 (VCC-)
- new net: R144.2, R152.2, U44.1
- new net: C38.2, FB20.1, U42.1 (V_{DD1})
- new net: R125.1, U36.3
- new net: R125.2, R133.1
- new net: IC9.1 (OUT), R115.2, U42.3 (V_{IA})
- new net: IC9.3 (IN+), R115.1, R116.2
- new net: IC9.4 (IN-), R117.2
- new net: C37.1, FB19.1, IC9.5 (VCC+)
- new net: R173.2, R179.2, U53.1
- new net: R176.2, R183.1, U53.3
- new net: R186.2, R194.2, U57.1
- new net: IC6.1 (OUT), R69.2, U27.4 (VIB)
- new net: IC6.3 (IN+), R69.1, R74.2
- new net: IC6.4 (IN-), R75.2
- new net: C25.1, FB14.1, IC6.5 (VCC+)
- new net: R178.2, R185.1, U55.3
- new net: R185.2, R192.1
- new net: R183.2, R190.1
- new net: D6.1 (A1), R111.1, R74.1, R99.2, U28.3
- new net: C62.1, R160.1, R172.1, R193.1, U61.6 (VOUT)
- new net: R177.2, R184.1, U54.3
- new net: R184.2, R191.1
- new net: R140.2, R147.1
- new net: IC14.3 (IN+), R182.1, R188.2
- new net: IC14.4 (IN-), R193.2
- new net: C57.1, FB28.1, IC14.5 (VCC+)
- new net: R63.2, R67.2, U21.1
- new net: R72.1, U21.3
- new net: R83.2, R92.1, U26.3
- new net: R101.1, R92.2
- new net: R163.2, R166.2, U52.1
- new net: R189.2, R196.2, U59.1
- new net: D12.1 (A1), R159.1, R190.2, R197.1, U59.3
- new net: C59.1, R200.1, U60.1 (K), U61.4 (AVDD/AVREF)
- new net: R127.1, U38.3
- new net: R170.1, U52.3
- new net: R170.2, R178.1
- new net: R103.2, R93.2, U28.1
- new net: R105.2, R95.2, U30.1
- new net: C58.1, C58.2, FB29.1, U62.10 (V_{E2}), U62.16 (V_{DD2})
- new net: R126.1, U37.3
- new net: R126.2, R134.1
- new net: C27.1, FB16.1, IC8.5 (VCC+)
- new net: IC7.3 (IN+), R88.1, R96.2
- new net: IC7.1 (OUT), R88.2, U27.5 (VIC)
- new net: U47.1 (~{SYNC}), U48.12 (V_{OC})
- new net: U47.2 (SCLK), U48.13 (V_{OB})
- new net: U47.3 (DIN), U48.14 (V_{OA})
- new net: C44.1, R157.1, U46.1 (K), U47.4 (AVDD/AVREF)
- new net: C47.1, R117.1, R129.1, R150.1, U47.6 (VOUT)
- new net: R106.2, R97.2, U31.1
- new net: R72.2, R82.1
- new net: R80.2, R89.1, U23.3
- new net: D11.1 (A1), R145.1, R149.2, R156.1, U44.3
- new net: IC12.3 (IN+), R158.1, R159.2
- new net: IC5.4 (IN-), R60.2
- new net: R174.2, R180.2, U54.1
- new net: D5.1 (A1), R110.1, R59.1, R98.2, U31.3
- new net: R70.1, U19.3
- new net: R70.2, R80.1
- new net: R146.2, R153.2, U45.1
- new net: C43.1, C43.2, FB23.1, U48.10 (V_{E2}), U48.16 (V_{DD2})
- new net: C29.1, R114.1, U32.1 (K), U33.4 (AVDD/AVREF)
- new net: R175.2, R181.2, U55.1
- new net: C52.1, FB25.1, IC12.5 (VCC+)
- new net: C48.2, C49.1, FB25.2, FB26.2, FB27.2, FB28.2, FB29.2, FB30.2, U49.4 (+Vout)
- new net: IC8.3 (IN+), R107.1, R108.2
- new net: R134.2, R141.1, U40.3
- new net: IC11.1 (OUT), R139.2, U42.5 (V_{IC})
- new net: IC11.3 (IN+), R139.1, R145.2
- new net: IC11.4 (IN-), R150.2
- new net: C42.1, FB22.1, IC11.5 (VCC+)
- new net: R143.2, R151.2, U43.1
- new net: D13.1 (A1), R171.1, R191.2, R198.1, U57.3
- new net: R104.2, R94.2, U29.1
- new net: R62.2, R66.2, U20.1
- new net: R89.2, R98.1
- new net: R133.2, R140.1, U39.3
- new net: U33.1 (~{SYNC}), U34.12 (V_{OC})
- new net: U33.2 (SCLK), U34.13 (V_{OB})
- new net: U33.3 (DIN), U34.14 (V_{OA})
- new net: R130.2, R136.2, U39.1
- new net: R131.2, R137.2, U40.1
- new net: IC12.4 (IN-), R160.2
- new net: IC8.1 (OUT), R107.2, U27.6 (VID)
- new net: IC8.4 (IN-), R109.2
- new net: R169.2, R177.1
- new net: C26.1, FB15.1, IC7.5 (VCC+)
- new net: R127.2, R135.1
- new net: R82.2, R91.1, U25.3
- new net: IC13.3 (IN+), R167.1, R171.2
- new net: IC10.1 (OUT), R124.2, U42.4 (V_{IB})
- new net: IC10.3 (IN+), R124.1, R128.2
- new net: IC10.4 (IN-), R129.2
- new net: C41.1, FB21.1, IC10.5 (VCC+)
- new net: FB18.1, R114.2
- new net: R100.1, R91.2
- new net: R161.2, R164.2, U50.1
- new net: R168.1, U50.3
- new net: R142.2, R149.1
- new net: IC13.4 (IN-), R172.2
- new net: R73.1, U22.3
- new net: R73.2, R83.1
- new net: R71.2, R81.1
- new net: R81.2, R90.1, U24.3
- new net: R79.2, R87.2, U26.1
- new net: D10.1 (A1), R128.1, R148.2, R155.1, U43.3
- new net: FB30.1, R200.2
- new net: R61.2, R65.2, U19.1
- new net: R118.2, R121.2, U36.1
- new net: R64.2, R68.2, U22.1
- new net: U61.1 (~{SYNC}), U62.12 (V_{OC})
- new net: U61.2 (SCLK), U62.13 (V_{OB})
- new net: U61.3 (DIN), U62.14 (V_{OA})
- new net: IC7.4 (IN-), R102.2
- new net: C22.2, FB13.1, U27.1 (VDD1)
- new net: R187.2, R195.2, U58.1
- new net: D7.1 (A1), R100.2, R112.1, R96.1, U29.3
- new net: R77.2, R85.2, U24.1
- new net: R71.1, U20.3
- new net: R90.2, R99.1
- new net: R168.2, R176.1
- new net: R78.2, R86.2, U25.1
- new net: R141.2, R148.1
- new net: C28.1, C28.2, FB17.1, U34.10 (V_{E2}), U34.16 (V_{DD2})
- new net CH2_IN1_R15: R84.1, U23.2
- new net CH2_IN1_R25: R65.1, U19.2
- new net CH2_IN1_R5: R106.1, U31.2
- new net CH2_IN2_R15: R85.1, U24.2
- new net CH2_IN2_R25: R66.1, U20.2
- new net CH2_IN2_R5: R103.1, U28.2
- new net CH2_IN3_R15: R86.1, U25.2
- new net CH2_IN3_R25: R67.1, U21.2
- new net CH2_IN3_R5: R104.1, U29.2
- new net CH2_IN4_R15: R87.1, U26.2
- new net CH2_IN4_R25: R68.1, U22.2
- new net CH2_IN4_R5: R105.1, U30.2
- new net CH3_IN1_R15: R136.1, R179.1, U39.2, U53.2
- new net CH3_IN1_R25: R121.1, R164.1, U36.2, U50.2
- new net CH3_IN1_R5: R153.1, R196.1, U45.2, U59.2
- new net CH3_IN2_R15: R137.1, R180.1, U40.2, U54.2
- new net CH3_IN2_R25: R122.1, R165.1, U37.2, U51.2
- new net CH3_IN2_R5: R151.1, R194.1, U43.2, U57.2
- new net CH3_IN3_R15: R138.1, R181.1, U41.2, U55.2
- new net CH3_IN3_R25: R123.1, R166.1, U38.2, U52.2
- new net CH3_IN3_R5: R152.1, R195.1, U44.2, U58.2
- new net DAC_CS2: U34.5 (V_{IC})
- new net DAC_CS3: U48.5 (V_{IC})
- new net DAC_CS4: U62.5 (V_{IC})
Other:
- moved on the sheet: C1, C10, C11, C12, C13, C14, C15, C16, C2, C4, C5, C6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

Commit message: Update TSC_board schematic and layout
Connections:
- net at C48.1, C49.2, C53.1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: now also C52.2, C56.2, C57.2, D12.2 (A2), D13.2 (A2), D14.2 (A2), IC12.2 (VCC-), IC13.2 (VCC-), IC14.2 (VCC-), J4.4 (Pin_4), R197.2, R198.2, R199.2
- net at C17.1, C18.2, C22.1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: now also C21.2, C25.2, C26.2, C27.2, D5.2 (A2), D6.2 (A2), D7.2 (A2), D8.2 (A2), IC5.2 (VCC-), IC6.2 (VCC-), IC7.2 (VCC-), IC8.2 (VCC-), J2.5 (Pin_5), R110.2, R111.2, R112.2, R113.2
- net at C10.2, C11.2, C5.2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: now also C1.1, C13.2, C16.2, C2.2, C6.1, U1.3 (-Vout), U10.2 (GND1), U10.8 (GND1), U15.2 (A), U16.5 (GND), U17.15 (GND_{2}), U17.9 (GND_{2})
- net at C37.2, C41.2, C42.2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: now also C33.1, C34.2, C38.1, C43.2, C44.2, C47.2, J3.4 (Pin_4), R154.2, R155.2, R156.2, U35.3 (-Vout), U42.2 (GND_{1}), U42.8 (GND_{1}), U46.2 (A), U47.5 (GND), U48.15 (GND_{2}), U48.9 (GND_{2})
- net at C43.1, FB23.1, U48.10 (V_{E2})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: no longer C43.2
Changed lines of the file:
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@@
 	)
 	(junction
+		(at 510.54 123.19)
+		(diameter 0)
+		(color 0 0 0 0)
+	)
+	(junction
 		(at 260.35 62.23)
 		(diameter 0)
@@
 	)
 	(junction
+		(at 444.5 516.89)
+		(diameter 0)
+		(color 0 0 0 0)
+	)
+	(junction
 		(at 584.2 77.47)
 		(diameter 0)
@@
 	)
 	(junction
+		(at 510.54 386.08)
+		(diameter 0)
+		(color 0 0 0 0)
+	)
+	(junction
 		(at 260.35 194.31)
 		(diameter 0)
@@
 	)
 	(junction
-		(at 548.64 411.48)
-		(diameter 0)
-		(color 0 0 0 0)
-	)
-	(junction
 		(at 373.38 194.31)
 		(diameter 0)
@@
 	)
 	(junction
+		(at 510.54 265.43)
+		(diameter 0)
+		(color 0 0 0 0)
+	)
+	(junction
 		(at 458.47 77.47)
 		(diameter 0)
@@
 	)
 	(junction
+		(at 551.18 252.73)
+		(diameter 0)
+		(color 0 0 0 0)
+	)
+	(junction
 		(at 203.2 233.68)
 		(diameter 0)
@@
 	)
 	(junction
+		(at 551.18 107.95)
+		(diameter 0)
+		(color 0 0 0 0)
+	)
+	(junction
 		(at 354.33 490.22)
 		(diameter 0)
@@
 	)
 	(junction
+		(at 419.1 539.75)
+		(diameter 0)
+		(color 0 0 0 0)
+	)
+	(junction
 		(at 551.18 438.15)
 		(diameter 0)
@@
 	)
 	(junction
+		(at 419.1 408.94)
+		(diameter 0)
+		(color 0 0 0 0)
+	)
+	(junction
 		(at 375.92 356.87)
 		(diameter 0)
@@
 	)
 	(junction
+		(at 444.5 386.08)
+		(diameter 0)
+		(color 0 0 0 0)
+	)
+	(junction
 		(at 508 260.35)
 		(diameter 0)
@@
 	)
 	(junction
+		(at 510.54 516.89)
+		(diameter 0)
+		(color 0 0 0 0)
+	)
+	(junction
 		(at 476.25 219.71)
 		(diameter 0)
@@
 	)
 	(junction
+		(at 551.18 411.48)
+		(diameter 0)
+		(color 0 0 0 0)
+	)
+	(junction
 		(at 510.54 67.31)
 		(diameter 0)
@@
 	(wire
 		(pts
+			(xy 538.48 252.73) (xy 551.18 252.73)
+		)
+		(stroke
+			(width 0)
+			(type default)
+		)
+	)
+	(wire
+		(pts
 			(xy 411.48 46.99) (xy 411.48 54.61)
 		)
@@
 	(wire
 		(pts
+			(xy 444.5 408.94) (xy 444.5 386.08)
+		)
+		(stroke
+			(width 0)
+			(type default)
+		)
+	)
+	(wire
+		(pts
 			(xy 260.35 222.25) (xy 260.35 223.52)
 		)
@@
 	(wire
 		(pts
+			(xy 551.18 411.48) (xy 554.99 411.48)
+		)
+		(stroke
+			(width 0)
+			(type default)
+		)
+	)
+	(wire
+		(pts
 			(xy 377.19 204.47) (xy 391.16 204.47)
 		)
@@
 	(wire
 		(pts
+			(xy 551.18 411.48) (xy 551.18 438.15)
+		)
+		(stroke
+			(width 0)
+			(type default)
+		)
+	)
+	(wire
+		(pts
 			(xy 495.3 245.11) (xy 508 245.11)
 		)
@@
 	(wire
 		(pts
-			(xy 551.18 100.33) (xy 551.18 166.37)
+			(xy 551.18 100.33) (xy 551.18 107.95)
 		)
 		(stroke
@@
 	(wire
 		(pts
-			(xy 554.99 411.48) (xy 548.64 411.48)
-		)
-		(stroke
-			(width 0)
-			(type default)
-		)
-	)
-	(wire
-		(pts
 			(xy 551.18 339.09) (xy 552.45 339.09)
 		)
@@
 	(wire
 		(pts
+			(xy 419.1 539.75) (xy 444.5 539.75)
+		)
+		(stroke
+			(width 0)
+			(type default)
+		)
+	)
+	(wire
+		(pts
 			(xy 473.71 48.26) (xy 477.52 48.26)
 		)
@@
 	(wire
 		(pts
+			(xy 538.48 107.95) (xy 551.18 107.95)
+		)
+		(stroke
+			(width 0)
+			(type default)
+		)
+	)
+	(wire
+		(pts
 			(xy 551.18 358.14) (xy 557.53 358.14)
 		)
@@
 	(wire
 		(pts
+			(xy 510.54 123.19) (xy 538.48 123.19)
+		)
+		(stroke
+			(width 0)
+			(type default)
+		)
+	)
+	(wire
+		(pts
 			(xy 394.97 516.89) (xy 397.51 516.89)
 		)
@@
 	(wire
 		(pts
+			(xy 538.48 123.19) (xy 538.48 107.95)
+		)
+		(stroke
+			(width 0)
+			(type default)
+		)
+	)
+	(wire
+		(pts
 			(xy 440.69 250.19) (xy 440.69 232.41)
 		)
@@
 	(wire
 		(pts
+			(xy 510.54 265.43) (xy 538.48 265.43)
+		)
+		(stroke
+			(width 0)
+			(type default)
+		)
+	)
+	(wire
+		(pts
 			(xy 323.85 194.31) (xy 323.85 196.85)
 		)
@@
 	(wire
 		(pts
-			(xy 551.18 386.08) (xy 551.18 438.15)
+			(xy 551.18 386.08) (xy 551.18 411.48)
 		)
 		(stroke
@@
 	(wire
 		(pts
+			(xy 538.48 265.43) (xy 538.48 252.73)
+		)
+		(stroke
+			(width 0)
+			(type default)
+		)
+	)
+	(wire
+		(pts
 			(xy 480.06 566.42) (xy 480.06 568.96)
 		)
@@
 	(wire
 		(pts
+			(xy 444.5 539.75) (xy 444.5 516.89)
+		)
+		(stroke
+			(width 0)
+			(type default)
+		)
+	)
+	(wire
+		(pts
 			(xy 562.61 193.04) (xy 563.88 193.04)
 		)
@@
 	(wire
 		(pts
+			(xy 419.1 408.94) (xy 444.5 408.94)
+		)
+		(stroke
+			(width 0)
+			(type default)
+		)
+	)
+	(wire
+		(pts
 			(xy 510.54 516.89) (xy 476.25 516.89)
 		)
@@
 	(wire
 		(pts
+			(xy 551.18 107.95) (xy 551.18 166.37)
+		)
+		(stroke
+			(width 0)
+			(type default)
+		)
+	)
+	(wire
+		(pts
 			(xy 419.1 485.14) (xy 419.1 486.41)
 		)
@@
 	(wire
 		(pts
+			(xy 510.54 386.08) (xy 551.18 386.08)
+		)
+		(stroke
+			(width 0)
+			(type default)
+		)
+	)
+	(wire
+		(pts
 			(xy 508 342.9) (xy 508 358.14)
 		)
@@
 	(wire
 		(pts
-			(xy 551.18 242.57) (xy 551.18 308.61)
+			(xy 551.18 242.57) (xy 551.18 252.73)
 		)
 		(stroke
@@
 	(wire
 		(pts
+			(xy 551.18 252.73) (xy 551.18 308.61)
+		)
+		(stroke
+			(width 0)
+			(type default)
+		)
+	)
+	(wire
+		(pts
 			(xy 504.19 568.96) (xy 551.18 568.96)
 		)
@@
 	(wire
 		(pts
-			(xy 548.64 400.05) (xy 548.64 411.48)
+			(xy 548.64 400.05) (xy 548.64 415.29)
 		)
 		(stroke
@@
 	(wire
 		(pts
+			(xy 510.54 516.89) (xy 551.18 516.89)
+		)
+		(stroke
+			(width 0)
+			(type default)
+		)
+	)
+	(wire
+		(pts
 			(xy 510.54 123.19) (xy 476.25 123.19)
 		)
@@
 	(wire
 		(pts
-			(xy 548.64 411.48) (xy 548.64 415.29)
-		)
-		(stroke
-			(width 0)
-			(type default)
-		)
-	)
-	(wire
-		(pts
 			(xy 554.99 532.13) (xy 554.99 530.86)
 		)
@@
 		(dnp no)
 		(property "Reference" "U41"
-			(at 406.4 345.44 0)
+			(at 406.4 353.06 0)
 			(effects
 				(font
@@
 		)
 		(property "Value" "GAQY212GS"
-			(at 406.4 347.98 0)
+			(at 406.4 355.6 0)
 			(effects
 				(font
