File: pcb/Frontend.kicad_sch (KiCad schematic)
At the start: 418 parts, among them IC1 TS3021ILT, IC10 TS3021ILT, IC11 TS3021ILT, IC12 TS3021ILT, IC13 TS3021ILT, IC14 TS3021ILT, IC15 NCP51460SN33T1G, IC16 NCP51460SN33T1G, IC17 NCP51460SN33T1G, IC18 NCP51460SN33T1G, IC2 TS3021ILT, IC3 TS3021ILT, IC4 TS3021ILT, IC5 TS3021ILT, IC6 TS3021ILT, IC7 TS3021ILT, IC8 TS3021ILT, IC9 TS3021ILT, J1 Conn_01x05_Socket, J2 Conn_01x05_Socket, J3 Conn_01x04_Socket, J4 Conn_01x04_Socket, U1 TEA1-0505, U10 ADuM1400xRW, U11 GAQY212GS, U12 GAQY212GS, U13 GAQY212GS, U14 GAQY212GS, U15 LM4040DBZ-5, U16 DAC7311xDCK, U17 ADuM1300xRW, U18 TEA1-0505, U19 GAQY212GS, U2 GAQY212GS, U20 GAQY212GS, U21 GAQY212GS, U22 GAQY212GS, U23 GAQY212GS, U24 GAQY212GS, U25 GAQY212GS, U26 GAQY212GS, U27 ADuM1400xRW, U28 GAQY212GS, U29 GAQY212GS, U3 GAQY212GS, U30 GAQY212GS, U31 GAQY212GS, U32 LM4040DBZ-5, U33 DAC7311xDCK, U34 ADuM1300xRW, U35 TEA1-0505, U36 GAQY212GS, U37 GAQY212GS, U38 GAQY212GS, U39 GAQY212GS, U4 GAQY212GS, U40 GAQY212GS, U41 GAQY212GS, U42 ADuM1300xRW, U43 GAQY212GS, U44 GAQY212GS, U45 GAQY212GS, U46 LM4040DBZ-5, U47 DAC7311xDCK, U48 ADuM1300xRW, U49 TEA1-0505, U5 GAQY212GS, U50 GAQY212GS, U51 GAQY212GS, U52 GAQY212GS, U53 GAQY212GS, U54 GAQY212GS, U55 GAQY212GS, U56 ADuM1300xRW, U57 GAQY212GS, U58 GAQY212GS, U59 GAQY212GS, U6 GAQY212GS, U60 LM4040DBZ-5, U61 DAC7311xDCK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

Commit message: Cleaning
Parts:
- removed TP1, TP2, TP5, TP6, TP8, TP9: TestPoint, TestPoint:TestPoint_Pad_D1.0mm, symbol Connector:TestPoint
- added TP13, TP14, TP15, TP16, TP17, TP18: TestPoint, TestPoint:TestPoint_Pad_D1.0mm, symbol Connector:TestPoint
- C1, C10, C11, C12, C13, C15, C17, C20, C21, C22, C24, C25, C26, C27, C28, C29, C31, C33, C36, C37, C38, C4, C40, C41, C42, C43, C44, C46, C48, C5, C51, C52, C53, C55, C56, C57, C58, C59, C6, C61, C64, C65, C66, C67, C68, C69, C70, C71, C8, C9: Manufacturer_Part_Number (none) -> GRM188R71H104KA93D
- C14, C19, C23, C3, C30, C35, C39, C45, C50, C54, C60, C7: Manufacturer_Part_Number (none) -> GRM1885C1H103JA01J
- C16, C32, C47, C62: Manufacturer_Part_Number (none) -> VJ0603A102JXACW1BC
- C18, C2, C34, C49: Manufacturer_Part_Number (none) -> CL31B106KBHNNNE
- D1, D10, D11, D12, D13, D14, D2, D3, D4, D5, D6, D7, D8, D9: Manufacturer_Part_Number (none) -> SMF5.0CA
- D15, D16, D17, D18: Manufacturer_Part_Number (none) -> 1N4148
- FB10, FB11, FB12, FB13, FB14, FB15, FB16, FB17, FB18, FB19, FB20, FB21, FB22, FB23, FB24, FB25, FB26, FB27, FB28, FB29, FB30, FB5, FB6, FB7, FB8, FB9: Manufacturer_Part_Number (none) -> WLBD1608HCU101TL
- J1, J2, J3, J4, TP10, TP11, TP12, TP3, TP4, TP7: now left out of the parts list
- R10, R100, R101, R103, R104, R105, R106, R11, R110, R111, R112, R113, R121, R122, R123, R125, R126, R127, R13, R133, R134, R135, R136, R137, R138, R14, R140, R141, R142, R147, R148, R149, R15, R151, R152, R153, R154, R155, R156, R16, R164, R165, R166, R168, R169, R170, R176, R177, R178, R179, R180, R181, R183, R184, R185, R190, R191, R192, R194, R195, R196, R197, R198, R199, R201, R202, R203, R204, R23, R24, R25, R26, R27, R28, R29, R30, R32, R33, R34, R35, R41, R42, R43, R44, R46, R47, R48, R49, R53, R54, R55, R56, R65, R66, R67, R68, R70, R71, R72, R73, R8, R80, R81, R82, R83, R84, R85, R86, R87, R89, R9, R90, R91, R92, R98, R99: Manufacturer_Part_Number (none) -> CRCW060310K0FKTABC
- R108, R116, R128, R145, R159, R17, R171, R188, R2, R39, R51, R59, R74, R96: Manufacturer_Part_Number (none) -> ERA3AEB2212V
- R114, R157, R200, R57: Manufacturer_Part_Number (none) -> 0603SAF3300T5E
- U1, U18, U35, U49: Manufacturer_Part_Number (none) -> TEA1-0505
- U10, U27: Manufacturer_Part_Number (none) -> ADuM1400BRW
- U11, U12, U13, U14, U19, U2, U20, U21, U22, U23, U24, U25, U26, U28, U29, U3, U30, U31, U36, U37, U38, U39, U4, U40, U41, U43, U44, U45, U5, U50, U51, U52, U53, U54, U55, U57, U58, U59, U6, U7, U8, U9: Manufacturer_Part_Number (none) -> GAQY212GS
- U15, U32, U46, U60: Manufacturer_Part_Number (none) -> LM4040DBZ-5
- U16, U33, U47, U61: Manufacturer_Part_Number (none) -> DAC7311IDCK
- U17, U34, U42, U48, U56, U62: Manufacturer_Part_Number (none) -> ADuM1300BRW
- U64, U65, U66, U67: Manufacturer_Part_Number (none) -> STM32C011F4P6
Connections:
- net at U64.18 (PA13): now also TP17.1
- net at U66.18 (PA13): now also TP13.1
- net at U65.18 (PA13): now also TP15.1
- net at U65.19 (PA14): now also TP16.1
- net at U64.19 (PA14): now also TP18.1
- net at U66.19 (PA14): now also TP14.1

Commit message: Update dac pwr
Parts:
- U15: now not fitted
- U32, U46, U60: value LM4040DBZ-5 -> LM4040D33FTA; now not fitted
Changed lines of the file:
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@@
 	)
 	(junction
+		(at 504.19 135.89)
+		(diameter 0)
+		(color 0 0 0 0)
+	)
+	(junction
 		(at 391.16 242.57)
 		(diameter 0)
@@
 	)
 	(junction
-		(at 504.19 166.37)
-		(diameter 0)
-		(color 0 0 0 0)
-	)
-	(junction
 		(at 458.47 232.41)
 		(diameter 0)
@@
 	)
 	(junction
-		(at 504.19 135.89)
-		(diameter 0)
-		(color 0 0 0 0)
-	)
-	(junction
 		(at 551.18 488.95)
 		(diameter 0)
@@
 	)
 	(junction
+		(at 504.19 166.37)
+		(diameter 0)
+		(color 0 0 0 0)
+	)
+	(junction
 		(at 276.86 508)
 		(diameter 0)
@@
 	(wire
 		(pts
-			(xy 504.19 144.78) (xy 504.19 166.37)
+			(xy 504.19 146.05) (xy 504.19 166.37)
 		)
 		(stroke
@@
 	(wire
 		(pts
-			(xy 504.19 137.16) (xy 504.19 135.89)
+			(xy 504.19 138.43) (xy 504.19 135.89)
 		)
 		(stroke
@@
 		(on_board yes)
 		(in_pos_files yes)
-		(dnp no)
+		(dnp yes)
 		(fields_autoplaced yes)
 		(property "Reference" "U60"
@@
 			)
 		)
-		(property "Value" "LM4040DBZ-5"
+		(property "Value" "LM4040D33FTA"
 			(at 506.73 544.8299 90)
 			(show_name no)
@@
 		(on_board yes)
 		(in_pos_files yes)
-		(dnp no)
+		(dnp yes)
 		(fields_autoplaced yes)
 		(property "Reference" "U46"
@@
 			)
 		)
-		(property "Value" "LM4040DBZ-5"
+		(property "Value" "LM4040D33FTA"
 			(at 506.73 414.0199 90)
 			(show_name no)
@@
 	(symbol
 		(lib_id "Reference_Voltage:LM4040DBZ-5")
-		(at 504.19 140.97 90)
+		(at 504.19 142.24 90)
 		(unit 1)
 		(body_style 1)
@@
 		(on_board yes)
 		(in_pos_files yes)
-		(dnp no)
+		(dnp yes)
 		(fields_autoplaced yes)
 		(property "Reference" "U15"
-			(at 506.73 139.6999 90)
+			(at 506.73 140.9699 90)
 			(show_name no)
 			(do_not_autoplace no)
@@
 		)
 		(property "Value" "LM4040DBZ-5"
-			(at 506.73 142.2399 90)
+			(at 506.73 143.5099 90)
 			(show_name no)
 			(do_not_autoplace no)
@@
 		)
 		(property "Footprint" "Package_TO_SOT_SMD:SOT-23"
-			(at 509.27 140.97 0)
+			(at 509.27 142.24 0)
 			(hide yes)
 			(show_name no)
@@
 		)
 		(property "Datasheet" "http://www.ti.com/lit/ds/symlink/lm4040-n.pdf"
-			(at 504.19 140.97 0)
+			(at 504.19 142.24 0)
 			(hide yes)
 			(show_name no)
@@
 		)
 		(property "Description" "5.000V Precision Micropower Shunt Voltage Reference, SOT-23"
-			(at 504.19 140.97 0)
+			(at 504.19 142.24 0)
 			(hide yes)
 			(show_name no)
@@
 		)
 		(property "Sim.Device" ""
-			(at 504.19 140.97 90)
+			(at 504.19 142.24 90)
 			(hide yes)
 			(show_name no)
@@
 		)
 		(property "Sim.Pins" ""
-			(at 504.19 140.97 90)
+			(at 504.19 142.24 90)
 			(hide yes)
 			(show_name no)
@@
 		)
 		(property "Manufacturer_Part_Number" "LM4040DBZ-5"
-			(at 504.19 140.97 90)
+			(at 504.19 142.24 90)
 			(hide yes)
 			(show_name no)
@@
 		(on_board yes)
 		(in_pos_files yes)
-		(dnp no)
+		(dnp yes)
 		(fields_autoplaced yes)
 		(property "Reference" "U32"
@@
 			)
 		)
-		(property "Value" "LM4040DBZ-5"
+		(property "Value" "LM4040D33FTA"
 			(at 506.73 284.4799 90)
 			(show_name no)

Commit message: Unify passive values, fix LM4040 DNP value, refresh outputs
Parts:
- R114, R157, R200, R57: value 330R -> 330
- U15: value LM4040DBZ-5 -> LM4040D33FTA
Changed lines of the file:
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@@
 			)
 		)
-		(property "Value" "330R"
+		(property "Value" "330"
 			(at 513.08 274.32 90)
 			(show_name no)
@@
 			)
 		)
-		(property "Value" "LM4040DBZ-5"
+		(property "Value" "LM4040D33FTA"
 			(at 506.73 143.5099 90)
 			(show_name no)
@@
 			)
 		)
-		(property "Value" "330R"
+		(property "Value" "330"
 			(at 513.08 403.86 90)
 			(show_name no)
@@
 			)
 		)
-		(property "Value" "330R"
+		(property "Value" "330"
 			(at 513.08 534.67 90)
 			(show_name no)
@@
 			)
 		)
-		(property "Value" "330R"
+		(property "Value" "330"
 			(at 513.08 132.08 90)
 			(show_name no)

Commit message: Last fixes
Parts:
- U15, U32, U46, U60: Manufacturer_Part_Number LM4040DBZ-5 -> LM4040D33FTA
Connections:
- net GND_ISO4: now reaches C48.1, C49.2, C52.2, C53.1, C56.2, C57.2, C58.2, C59.2, C62.2, D12.2 (A2), D13.2 (A2), D14.2 (A2), IC12.2 (VCC-), IC13.2 (VCC-), IC14.2 (VCC-), J4.4 (Pin_4), R197.2, R198.2, R199.2, U49.3 (-Vout), U56.2 (GND_{1}), U56.8 (GND_{1}), U60.2 (A), U61.5 (GND), U62.15 (GND_{2}), U62.9 (GND_{2})
- net GND_ISO2: now reaches C17.1, C18.2, C21.2, C22.1, C25.2, C26.2, C27.2, C28.2, C29.2, C32.2, D5.2 (A2), D6.2 (A2), D7.2 (A2), D8.2 (A2), IC5.2 (VCC-), IC6.2 (VCC-), IC7.2 (VCC-), IC8.2 (VCC-), J2.5 (Pin_5), R110.2, R111.2, R112.2, R113.2, U18.3 (-Vout), U27.2 (GND1), U27.8 (GND1), U32.2 (A), U33.5 (GND), U34.15 (GND_{2}), U34.9 (GND_{2})
- net +5V_ISO2: now reaches C17.2, C18.1, FB12.2, FB13.2, FB14.2, FB15.2, FB16.2, FB17.2, FB18.2, U18.4 (+Vout)
- net GND_ISO1: now reaches C1.1, C10.2, C11.2, C12.2, C13.2, C16.2, C2.2, C5.2, C6.1, C9.2, D1.2 (A2), D2.2 (A2), D3.2 (A2), D4.2 (A2), IC1.2 (VCC-), IC2.2 (VCC-), IC3.2 (VCC-), IC4.2 (VCC-), J1.5 (Pin_5), R53.2, R54.2, R55.2, R56.2, U1.3 (-Vout), U10.2 (GND1), U10.8 (GND1), U15.2 (A), U16.5 (GND), U17.15 (GND_{2}), U17.9 (GND_{2})
- net +5V_ISO1: now reaches C1.2, C2.1, FB10.2, FB11.2, FB5.2, FB6.2, FB7.2, FB8.2, FB9.2, U1.4 (+Vout)
- net +5V_ISO3: now reaches C33.2, C34.1, FB19.2, FB20.2, FB21.2, FB22.2, FB23.2, FB24.2, U35.4 (+Vout)
- net GND_ISO3: now reaches C33.1, C34.2, C37.2, C38.1, C41.2, C42.2, C43.2, C44.2, C47.2, D10.2 (A2), D11.2 (A2), D9.2 (A2), IC10.2 (VCC-), IC11.2 (VCC-), IC9.2 (VCC-), J3.4 (Pin_4), R154.2, R155.2, R156.2, U35.3 (-Vout), U42.2 (GND_{1}), U42.8 (GND_{1}), U46.2 (A), U47.5 (GND), U48.15 (GND_{2}), U48.9 (GND_{2})
- net +5V_ISO4: now reaches C48.2, C49.1, FB25.2, FB26.2, FB27.2, FB28.2, FB29.2, FB30.2, U49.4 (+Vout)

Commit message: Fix BOM data: 1k resistor MPN, 1N4148WS diodes, ADuM/DAC7311 orderable part numbers, BOM export settings
Parts:
- D15, D16, D17, D18: Manufacturer_Part_Number 1N4148 -> 1N4148WS
- J1, J2: Manufacturer_Part_Number (none) -> OQ0512510000G; now in the parts list
- J3, J4: Manufacturer_Part_Number (none) -> 15EDGRC-3.5/4P; now in the parts list
- R108, R116, R128, R145, R159, R17, R171, R188, R2, R39, R51, R59, R74, R96: Manufacturer_Part_Number ERA3AEB2212V -> (none)
- U10, U27: value ADuM1400xRW -> ADuM1400BRWZ
- U16, U33, U47, U61: value DAC7311xDCK -> DAC7311IDCKR
- U17, U34, U42, U48, U56, U62: value ADuM1300xRW -> ADuM1300BRWZ
- U64, U65, U66, U67: value STM32C011F4Px -> STM32C011F4P6
