File: pcb/Conn.kicad_sch (KiCad schematic)
At the start: 5 parts

Commit message: Before DRC
Connections:
- net UART_RX: now reaches X1.32 (PB6)
- net UART_TX: now reaches X1.33 (PB5)
Changed lines of the file:
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@@
+	(wire
+		(pts
+			(xy 214.63 88.9) (xy 218.44 88.9)
+		)
+		(stroke
+			(width 0)
+			(type default)
+		)
+	)
 	(wire
 		(pts
@@
 	(wire
 		(pts
+			(xy 237.49 86.36) (xy 241.3 86.36)
+		)
+		(stroke
+			(width 0)
+			(type default)
+		)
+	)
+	(wire
+		(pts
 			(xy 237.49 104.14) (xy 241.3 104.14)
 		)
@@
 		)
 	)
+	(hierarchical_label "UART_RX"
+		(shape input)
+		(at 241.3 86.36 0)
+		(effects
+			(font
+				(size 1.27 1.27)
+			)
+			(justify left)
+		)
+	)
 	(hierarchical_label "QSPI_IO0"
 		(shape input)
@@
 		)
 	)
+	(hierarchical_label "UART_TX"
+		(shape input)
+		(at 214.63 88.9 180)
+		(effects
+			(font
+				(size 1.27 1.27)
+			)
+			(justify right)
+		)
+	)
